File: hardware/project/ADC_Test/Connector.sch (KiCad schematic (older format))
At the start: 1 part, among them J601 C64AC

Commit message: Schematic design.
Parts:
- renumbered J601 to J301
Connections:
- net V_LOW: now also J301.A5 (5A), J301.C5 (5C); no longer J301.A3 (3A), J301.C3 (3C)
Changed lines of the file:
@@
 	5350 5050 5400 5050
 $Comp
-L power:Earth #PWR0602
+L power:Earth #PWR0302
 U 1 1 5DECE77F
 P 5350 5050
-F 0 "#PWR0602" H 5350 4800 50  0001 C CNN
+F 0 "#PWR0302" H 5350 4800 50  0001 C CNN
 F 1 "Earth" H 5350 4900 50  0001 C CNN
 F 2 "" H 5350 5050 50  0001 C CNN
@@
 	5450 5000 5400 5000
 Wire Wire Line
-	5400 1250 5400 1200
-Connection ~ 5400 1250
+	5400 1650 5400 1600
+Connection ~ 5400 1650
 Wire Wire Line
 	5400 1050 5400 1000
 Connection ~ 5400 1050
 Wire Wire Line
-	5400 1250 5200 1250
+	5400 1650 5200 1650
 Wire Wire Line
-	5400 1200 5450 1200
+	5400 1600 5450 1600
 Wire Wire Line
-	5400 1300 5400 1250
+	5400 1700 5400 1650
 Wire Wire Line
-	5450 1300 5400 1300
+	5450 1700 5400 1700
 Wire Wire Line
 	5400 1000 5450 1000
@@
 	5450 7100 5400 7100
 $Comp
-L Connector:C64AC J601
+L Connector:C64AC J301
 U 1 1 5DE8758D
 P 5750 4000
-F 0 "J601" H 5930 4096 50  0000 L CNN
+F 0 "J301" H 5930 4096 50  0000 L CNN
 F 1 "C64AC" H 5930 4005 50  0000 L CNN
 F 2 "ADC_TEST:Socket_DIN41612-CaseC1-AC-Male-64Pin-2rows" H 5750 4050 50  0001 C CNN
@@
 $EndComp
 $Comp
-L ADC_TEST:+24VF #PWR0604
+L ADC_TEST:+24VF #PWR0304
 U 1 1 60AC1A06
 P 5350 6950
-F 0 "#PWR0604" H 5350 6800 50  0001 C CNN
+F 0 "#PWR0304" H 5350 6800 50  0001 C CNN
 F 1 "+24VF" V 5365 7077 50  0000 L CNN
 F 2 "" H 5350 6950 50  0001 C CNN
@@
 $EndComp
 $Comp
-L ADC_TEST:DGNDF #PWR0603
+L ADC_TEST:DGNDF #PWR0303
 U 1 1 60AC7E80
 P 5350 6150
-F 0 "#PWR0603" H 5350 5900 50  0001 C CNN
+F 0 "#PWR0303" H 5350 5900 50  0001 C CNN
 F 1 "DGNDF" V 5355 6023 50  0000 R CNN
 F 2 "" H 5350 6150 50  0001 C CNN
@@
 NoConn ~ 5450 1400
 NoConn ~ 5450 1500
-NoConn ~ 5450 1600
-NoConn ~ 5450 1700
 NoConn ~ 5450 1800
 NoConn ~ 5450 1900
@@
 Text HLabel 5200 1050 0    50   Output ~ 0
 V_HIGH
-Text HLabel 5200 1250 0    50   Output ~ 0
+Text HLabel 5200 1650 0    50   Output ~ 0
 V_LOW
 Wire Wire Line
@@
 	5400 4300 5450 4300
 $Comp
-L power:Earth #PWR0601
+L power:Earth #PWR0301
 U 1 1 5DED2C4C
 P 5350 4250
-F 0 "#PWR0601" H 5350 4000 50  0001 C CNN
+F 0 "#PWR0301" H 5350 4000 50  0001 C CNN
 F 1 "Earth" H 5350 4100 50  0001 C CNN
 F 2 "" H 5350 4250 50  0001 C CNN
@@
 Wire Wire Line
 	5400 4250 5400 4300
+NoConn ~ 5450 1200
+NoConn ~ 5450 1300
 $EndSCHEMATC
