File: hardware/project/ADC_Test/Ethernet.sch (KiCad schematic (older format))
At the start: 43 parts, among them U701 LAN8742A, U702 LC03-3.3, U703 LC03-3.3, Y701 NX5032GA-25.000M-LN-CD-1

Commit message: Schematic design.
Parts:
- renumbered C701 to C401, C702 to C402, C703 to C403, C704 to C404, C705 to C405, C706 to C406, C707 to C407, C708 to C408, C709 to C409, C710 to C410, C711 to C411, C712 to C412, C713 to C413, C714 to C414, D701 to D401, D702 to D402, FB701 to FB401, L701 to L401, R701 to R401, R702 to R402, R703 to R403, R704 to R404, R705 to R405, R706 to R406, R707 to R407, R708 to R408, R709 to R409, R710 to R410, R711 to R411, R712 to R412, R713 to R413, R714 to R414, R715 to R415, R716 to R416, R717 to R417, R718 to R418, R719 to R419, R720 to R420, R721 to R421, U701 to U401, U702 to U402, U703 to U403, Y701 to Y401
