File: hardware/project/ADC_Test/FPGA.sch (KiCad schematic (older format))
At the start: 66 parts, among them J501 Conn_02x05, Q701 BC857W, U501 SN74LVC1T45DBV, U502 SN74LVC1T45DBV, U503 ICE40HX4K-TQ144, U504 SN74LVC1T45DBV, U505 SN74LVC1T45DBV, U506 SN74LVC1T45DBV, U507 SN74LVC1T45DBV, U508 ASDMB-100.000MHZ, U509 MT25QL128ABA1ESE

Commit message: Schematic design.
Parts:
- added J801: Conn_01x04_Male, Connector_PinHeader_2.54mm:PinHeader_1x04_P2.54mm_Vertical, symbol Connector:Conn_01x04_Male
- J802: renamed from J501; footprint Connector_PinHeader_2.54mm:PinHeader_2x05_P2.54mm_Vertical -> Connector_PinHeader_2.54mm:PinHeader_1x04_P2.54mm_Vertical
- R809: renamed from R722; footprint (none) -> Resistor_SMD:R_0603_1608Metric_Pad1.05x0.95mm_HandSolder
- renumbered C501 to C801, C502 to C802, C503 to C803, C504 to C804, C505 to C805, C506 to C806, C507 to C807, C508 to C808, C509 to C809, C510 to C810, C511 to C811, C512 to C812, C513 to C813, C514 to C814, C515 to C815, C516 to C816, C517 to C817, C518 to C818, C519 to C819, C520 to C820, C521 to C821, C522 to C822, C523 to C823, C524 to C824, C525 to C825, C526 to C826, C527 to C827, C528 to C828, C529 to C829, C530 to C830, C531 to C831, C532 to C832, D501 to D801, D502 to D802, D503 to D803, Q701 to Q801, R501 to R801, R502 to R802, R503 to R803, R504 to R804, R505 to R805, R506 to R806, R508 to R807, R509 to R808, R510 to R810, R511 to R811, R512 to R812, R513 to R813, R514 to R814, R515 to R815, R516 to R816, R517 to R817, R518 to R818, R519 to R819, R520 to R820, U501 to U801, U502 to U802, U503 to U803, U504 to U804, U505 to U805, U506 to U806, U507 to U807, U508 to U808, U509 to U809
Connections:
- net labels added: AD_IRP, AD_VRH, FGPA_AD_VRH
- net labels removed: FGPA_SW_VRH, SW_IRP, SW_VRH
- wire segments 288 -> 297
- no-connect marks 83 -> 79

Commit message: Schematic, PCB and BOM.
Parts:
- removed Q801: BC857W, Package_TO_SOT_SMD:SOT-323_SC-70, symbol Transistor_BJT:BC857W
- added Q801: BC857, Package_TO_SOT_SMD:SOT-23, symbol Transistor_BJT:BC857
- J802: footprint Connector_PinHeader_2.54mm:PinHeader_1x04_P2.54mm_Vertical -> Connector_PinHeader_2.54mm:PinHeader_2x05_P2.54mm_Vertical
Changed lines of the file:
@@
 F 0 "J802" H 15100 1817 50  0000 C CNN
 F 1 "Conn_02x05" H 15100 1726 50  0000 C CNN
-F 2 "Connector_PinHeader_2.54mm:PinHeader_1x04_P2.54mm_Vertical" H 15050 1400 50  0001 C CNN
+F 2 "Connector_PinHeader_2.54mm:PinHeader_2x05_P2.54mm_Vertical" H 15050 1400 50  0001 C CNN
 F 3 "~" H 15050 1400 50  0001 C CNN
 	1    15050 1400
@@
 Wire Wire Line
 	8050 1400 8100 1400
-$Comp
-L Transistor_BJT:BC857W Q801
-U 1 1 60B62038
-P 7500 1400
-F 0 "Q801" H 7691 1354 50  0000 L CNN
-F 1 "BC857W" H 7691 1445 50  0000 L CNN
-F 2 "Package_TO_SOT_SMD:SOT-323_SC-70" H 7700 1325 50  0001 L CIN
-F 3 "http://www.infineon.com/dgdl/Infineon-BC857SERIES_BC858SERIES_BC859SERIES_BC860SERIES-DS-v01_01-en.pdf?fileId=db3a304314dca389011541da0e3a1661" H 7500 1400 50  0001 L CNN
-	1    7500 1400
-	-1   0    0    1
-$EndComp
 Wire Wire Line
 	7700 1400 7750 1400
@@
 Wire Wire Line
 	5900 1400 5600 1400
+$Comp
+L Transistor_BJT:BC857 Q801
+U 1 1 5F8FD599
+P 7500 1400
+F 0 "Q801" H 7691 1354 50  0000 L CNN
+F 1 "BC857" H 7691 1445 50  0000 L CNN
+F 2 "Package_TO_SOT_SMD:SOT-23" H 7700 1325 50  0001 L CIN
+F 3 "http://www.fairchildsemi.com/ds/BC/BC856.pdf" H 7500 1400 50  0001 L CNN
+	1    7500 1400
+	-1   0    0    1
+$EndComp
 $EndSCHEMATC

Commit message: Changes in documentation, schematics and PCB.
Connections:
- net FPGA_AD_RFS_OPT: now reaches U803.39 (IOB_61)
- no-connect marks 79 -> 78
Other:
- moved on the sheet: Q801, R809
Changed lines of the file:
@@
 NoConn ~ 1850 3800
 NoConn ~ 1850 3900
-NoConn ~ 8100 1600
 NoConn ~ 8100 1700
 NoConn ~ 8100 1800
@@
 L Device:R R809
 U 1 1 60B17B60
-P 7900 1400
-F 0 "R809" V 8107 1400 50  0000 C CNN
-F 1 "6k2" V 8016 1400 50  0000 C CNN
-F 2 "Resistor_SMD:R_0603_1608Metric_Pad1.05x0.95mm_HandSolder" V 7830 1400 50  0001 C CNN
-F 3 "~" H 7900 1400 50  0001 C CNN
-	1    7900 1400
+P 7750 1400
+F 0 "R809" V 7957 1400 50  0000 C CNN
+F 1 "6k2" V 7866 1400 50  0000 C CNN
+F 2 "Resistor_SMD:R_0603_1608Metric_Pad1.05x0.95mm_HandSolder" V 7680 1400 50  0001 C CNN
+F 3 "~" H 7750 1400 50  0001 C CNN
+	1    7750 1400
 	0    -1   -1   0
 $EndComp
 Wire Wire Line
-	8050 1400 8100 1400
-Wire Wire Line
-	7700 1400 7750 1400
+	7500 1400 7600 1400
 $Comp
 L ADC_TEST:+3.3VF #PWR0830
 U 1 1 60B7C21D
-P 7400 1150
-F 0 "#PWR0830" H 7400 1000 50  0001 C CNN
-F 1 "+3.3VF" H 7415 1323 50  0000 C CNN
-F 2 "" H 7400 1150 50  0001 C CNN
-F 3 "" H 7400 1150 50  0001 C CNN
-	1    7400 1150
-	1    0    0    -1
-$EndComp
-Wire Wire Line
-	7400 1150 7400 1200
-Text HLabel 7400 1650 3    50   Output ~ 0
+P 7200 1150
+F 0 "#PWR0830" H 7200 1000 50  0001 C CNN
+F 1 "+3.3VF" H 7215 1323 50  0000 C CNN
+F 2 "" H 7200 1150 50  0001 C CNN
+F 3 "" H 7200 1150 50  0001 C CNN
+	1    7200 1150
+	1    0    0    -1
+$EndComp
+Wire Wire Line
+	7200 1150 7200 1200
+Text HLabel 7200 1650 3    50   Output ~ 0
 FPGA_AD_RFS
 Wire Wire Line
-	7400 1650 7400 1600
+	7200 1650 7200 1600
 Wire Wire Line
 	11850 6700 12450 6700
@@
 L Transistor_BJT:BC857 Q801
 U 1 1 5F8FD599
-P 7500 1400
-F 0 "Q801" H 7691 1354 50  0000 L CNN
-F 1 "BC857" H 7691 1445 50  0000 L CNN
-F 2 "Package_TO_SOT_SMD:SOT-23" H 7700 1325 50  0001 L CIN
-F 3 "http://www.fairchildsemi.com/ds/BC/BC856.pdf" H 7500 1400 50  0001 L CNN
-	1    7500 1400
+P 7300 1400
+F 0 "Q801" H 7491 1354 50  0000 L CNN
+F 1 "BC857" H 7491 1445 50  0000 L CNN
+F 2 "Package_TO_SOT_SMD:SOT-23" H 7500 1325 50  0001 L CIN
+F 3 "http://www.fairchildsemi.com/ds/BC/BC856.pdf" H 7300 1400 50  0001 L CNN
+	1    7300 1400
 	-1   0    0    1
 $EndComp
+Text HLabel 8050 1600 0    50   Output ~ 0
+FPGA_AD_RFS_OPT
+Wire Wire Line
+	7900 1400 8100 1400
+Wire Wire Line
+	8050 1600 8100 1600
 $EndSCHEMATC

Commit message: PCB design
Parts:
- removed C811, C826: 100n, Capacitor_SMD:C_0603_1608Metric_Pad1.05x0.95mm_HandSolder, symbol Device:C
- removed R812: 22, Resistor_SMD:R_0603_1608Metric_Pad1.05x0.95mm_HandSolder, symbol Device:R
- renumbered C802 to C801, C804 to C802, C806 to C803, C808 to C804, C809 to C805, C810 to C806, C812 to C807, C813 to C808, C814 to C809, C815 to C810, C816 to C811, C817 to C812, C818 to C813, C819 to C814, C820 to C815, C821 to C816, C822 to C817, C823 to C818, C824 to C819, C825 to C820, C801 to C821, C803 to C822, C827 to C823, C805 to C824, C828 to C825, C807 to C826, C829 to C827, C830 to C828, C831 to C829, C832 to C830, R813 to R812, R814 to R813, R815 to R814, R816 to R815, R817 to R816, R818 to R817, R819 to R818, R820 to R819
Connections:
- net 100MHZ_OPT: no longer names the net of U803.61 (IOB_96)
- no-connect marks 78 -> 79
Other:
- moved on the sheet: C807, C808, C809, C810, C811, C812, C813, C814, C815, C816, C817, C818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

Commit message: PCB design.
Parts:
- renumbered R809 to R801, R805 to R802, R804 to R803, R803 to R804, R802 to R805, R801 to R807, R807 to R809
Connections:
- net +3.3VF is gone; now on net +3.3VP: Q801.2 (E)
- net FPGA_AD_RFS_OPT: now also U803.8 (IOL_4B); no longer U803.39 (IOB_61)
- net FPGA_IO1: now also U803.99 (IOR_152); no longer U803.102 (IOR_161)
- net FPGA_IO2: now also U803.98 (IOR_148); no longer U803.101 (IOR_160)
- net FPGA_SPI3_MISO: now also U803.105 (IOR_165); no longer U803.95 (IOR_144)
- net FPGA_SPI3_MOSI: now also U803.104 (IOR_164); no longer U803.96 (IOR_146)
- net FPGA_SPI3_NSS: now also U803.107 (IOR_167); no longer U803.91 (IOR_139)
- net FPGA_SPI3_SCK: now also U803.106 (IOR_166); no longer U803.73 (IOR_109)
- net FPGA_UART2_CTRL_TTL: now also U803.81 (IOR_117); no longer U803.98 (IOR_148)
- net FPGA_UART2_RX_TTL: now also U803.82 (IOR_118); no longer U803.97 (IOR_147)
- net FPGA_UART2_TX_TTL: now also U803.83 (IOR_119); no longer U803.99 (IOR_152)
- net at R806.1: now also U803.136 (IOT_214); no longer U803.7 (IOL_4A)
- net at R802.1: now also U803.110 (IOT_168); no longer U803.4 (IOL_3B)
- net at R803.1: now also U803.115 (IOT_172); no longer U803.3 (IOL_3A)
- net at R804.1: now also U803.121 (IOT_181); no longer U803.2 (IOL_2B)
- net at R805.1: now also U803.130 (IOT_206); no longer U803.1 (IOL_2A)
- net at R809.1: now also U803.38 (IOB_57); no longer U803.10 (IOL_5B)
- net at R807.1: now also U803.37 (IOB_56); no longer U803.9 (IOL_5A)
- net at J801.1 (Pin_1): now also U803.2 (IOL_2B); no longer U803.110 (IOT_168)
- net at U803.112 (IOT_169): no longer J801.2 (Pin_2)
- net at U803.113 (IOT_170): no longer J801.3 (Pin_3)
- net at U803.114 (IOT_171): no longer J801.4 (Pin_4)
- net at R801.2: now also U803.1 (IOL_2A); no longer U803.37 (IOB_56)
- new net: J801.2 (Pin_2), U803.3 (IOL_3A)
- new net: J801.3 (Pin_3), U803.4 (IOL_3B)
- new net: J801.4 (Pin_4), U803.7 (IOL_4A)
- new net FPGA_IO3: U803.102 (IOR_161)
- new net FPGA_IO4: U803.101 (IOR_160)
- no-connect marks 79 -> 77
Other:
- moved on the sheet: D801, D802, J801, Q801, R801, R802, R803, R804, R805, R806, R807, R809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
