File: hardware/project/ADC_Test/ADC.sch (KiCad schematic (older format))
At the start: 47 parts, among them Q801 BC847W, U401 DG211CJD, U402 LT5400-100k-100k, U403 OPA2192, U404 DG419xY, U406 LM399H, U408 LT5400-5k-1k, U412 LT5400-10k-10k, U801 OPA177, U802 OPA140, U803 OPA177, U804 OPA192, U805 LM311

Commit message: Schematic design.
Parts:
- removed R317: 1M, Resistor_SMD:R_0603_1608Metric_Pad1.05x0.95mm_HandSolder, symbol Device:R
- added C501, C502, C503, C504, C505, C507, C510, C511, C512, C513, C514, C516, C518, C519, C520, C521, C523, C524: 100n, Capacitor_SMD:C_0603_1608Metric_Pad1.05x0.95mm_HandSolder, symbol Device:C
- added R515: 400/.1%, Resistor_SMD:R_0603_1608Metric_Pad1.05x0.95mm_HandSolder, symbol Device:R
- C515: renamed from C801; footprint (none) -> Capacitor_SMD:C_0603_1608Metric_Pad1.05x0.95mm_HandSolder
- C517: renamed from C802; footprint (none) -> Capacitor_SMD:C_0603_1608Metric_Pad1.05x0.95mm_HandSolder
- C522: renamed from C803; footprint (none) -> Capacitor_SMD:C_0603_1608Metric_Pad1.05x0.95mm_HandSolder
- D501: renamed from D801; value BAV103 -> BAV21W; footprint (none) -> Diode_SMD:D_SOD-123
- D502: renamed from D802; value BAV103 -> BAV21W; footprint (none) -> Diode_SMD:D_SOD-123
- D503: renamed from D803; value BAV103 -> BAV21W; footprint (none) -> Diode_SMD:D_SOD-123
- R501: renamed from R801; footprint (none) -> Resistor_SMD:R_0603_1608Metric_Pad1.05x0.95mm_HandSolder
- R502: renamed from R802; footprint (none) -> Resistor_SMD:R_0603_1608Metric_Pad1.05x0.95mm_HandSolder
- R503: renamed from R803; footprint (none) -> Resistor_SMD:R_0603_1608Metric_Pad1.05x0.95mm_HandSolder
- R504: renamed from R804; footprint (none) -> Resistor_SMD:R_0603_1608Metric_Pad1.05x0.95mm_HandSolder
- R505: renamed from R404; value 62 -> 62/.1%
- R506: renamed from R805; footprint (none) -> Resistor_SMD:R_0603_1608Metric_Pad1.05x0.95mm_HandSolder
- R507: renamed from R806; footprint (none) -> Resistor_SMD:R_0603_1608Metric_Pad1.05x0.95mm_HandSolder
- R509: renamed from R807; value 12k -> 12k/.05%; footprint (none) -> Resistor_SMD:R_0603_1608Metric_Pad1.05x0.95mm_HandSolder
- R512: renamed from R808; value 63k -> 62k6/.1%; footprint (none) -> Resistor_SMD:R_0603_1608Metric_Pad1.05x0.95mm_HandSolder
- R513: renamed from R809; footprint (none) -> Resistor_SMD:R_0603_1608Metric_Pad1.05x0.95mm_HandSolder
- R514: renamed from R810; footprint (none) -> Resistor_SMD:R_0603_1608Metric_Pad1.05x0.95mm_HandSolder
- R517: renamed from R811; value 620 -> 620/.05%; footprint (none) -> Resistor_SMD:R_0603_1608Metric_Pad1.05x0.95mm_HandSolder
- R518: renamed from R812; value 3k9 -> 3k9/.05%; footprint (none) -> Resistor_SMD:R_0603_1608Metric_Pad1.05x0.95mm_HandSolder
- R519: renamed from R813; footprint (none) -> Resistor_SMD:R_0603_1608Metric_Pad1.05x0.95mm_HandSolder
- R520: renamed from R814; value 62 -> 62/.1%; footprint (none) -> Resistor_SMD:R_0603_1608Metric_Pad1.05x0.95mm_HandSolder
- R521: renamed from R815; value 39k -> 39k/.05%; footprint (none) -> Resistor_SMD:R_0603_1608Metric_Pad1.05x0.95mm_HandSolder
- R522: renamed from R816; value 3k9 -> 3k9/.05%; footprint (none) -> Resistor_SMD:R_0603_1608Metric_Pad1.05x0.95mm_HandSolder
- TP501: renamed from TP801; footprint (none) -> TestPoint:TestPoint_Loop_D2.60mm_Drill1.6mm_Beaded
- TP502: renamed from TP802; footprint (none) -> TestPoint:TestPoint_Loop_D2.60mm_Drill1.6mm_Beaded
- TP503: renamed from TP803; footprint (none) -> TestPoint:TestPoint_Loop_D2.60mm_Drill1.6mm_Beaded
- U501: renamed from U401; value DG211CJD -> DG211B; footprint (none) -> Package_SO:SOIC-16_3.9x9.9mm_P1.27mm; symbol ADC_TEST:DG211CJD -> ADC_TEST:DG211
- U507: renamed from U801; footprint (none) -> Package_SO:SOIC-8_3.9x4.9mm_P1.27mm
- U508: renamed from U802; footprint (none) -> Package_SO:SOIC-8_3.9x4.9mm_P1.27mm
- U509: renamed from U803; footprint (none) -> Package_SO:SOIC-8_3.9x4.9mm_P1.27mm
- U510: renamed from U804; footprint (none) -> Package_SO:SOIC-8_3.9x4.9mm_P1.27mm
- U512: renamed from U805; footprint (none) -> Package_SO:SOIC-8_3.9x4.9mm_P1.27mm
- renumbered C421 to C506, C415 to C508, C416 to C509, Q801 to Q501, R406 to R508, R408 to R510, R407 to R511, R410 to R516, U403 to U502, U404 to U503, U402 to U504, U406 to U505, U408 to U506, U412 to U511
Connections:
- net labels added: VREF_-7V
- net labels removed: VR_-7V
- wire segments 212 -> 293
Other:
- moved on the sheet: C515, D502, D503, R507, R510, R511, R512, R517, R518

Commit message: Schematic, PCB and BOM.
Parts:
- removed Q501: BC847W, Package_TO_SOT_SMD:SOT-323_SC-70, symbol Transistor_BJT:BC847W
- added Q501: BC847, Package_TO_SOT_SMD:SOT-23, symbol Transistor_BJT:BC847
Changed lines of the file:
@@
-	1    0    0    -1
-$EndComp
-$Comp
-L Transistor_BJT:BC847W Q501
-U 1 1 60387261
-P 2850 6550
-F 0 "Q501" H 3040 6596 50  0000 L CNN
-F 1 "BC847W" H 3040 6505 50  0000 L CNN
-F 2 "Package_TO_SOT_SMD:SOT-323_SC-70" H 3050 6475 50  0001 L CIN
-F 3 "http://www.infineon.com/dgdl/Infineon-BC847SERIES_BC848SERIES_BC849SERIES_BC850SERIES-DS-v01_01-en.pdf?fileId=db3a304314dca389011541d4630a1657" H 2850 6550 50  0001 L CNN
-	1    2850 6550
 	1    0    0    -1
 $EndComp
@@
 Wire Wire Line
 	10900 10300 11100 10300
+$Comp
+L Transistor_BJT:BC847 Q501
+U 1 1 5F8DE25D
+P 2850 6550
+F 0 "Q501" H 3041 6596 50  0000 L CNN
+F 1 "BC847" H 3041 6505 50  0000 L CNN
+F 2 "Package_TO_SOT_SMD:SOT-23" H 3050 6475 50  0001 L CIN
+F 3 "http://www.infineon.com/dgdl/Infineon-BC847SERIES_BC848SERIES_BC849SERIES_BC850SERIES-DS-v01_01-en.pdf?fileId=db3a304314dca389011541d4630a1657" H 2850 6550 50  0001 L CNN
+	1    2850 6550
+	1    0    0    -1
+$EndComp
 $EndSCHEMATC

Commit message: Changes in documentation, schematics and PCB.
Parts:
- added C525: 10p, Capacitor_SMD:C_0603_1608Metric_Pad1.05x0.95mm_HandSolder, symbol Device:C
- added D504: BZT585B15TQ-13, Diode_SMD:D_SOD-523, symbol Device:D_Zener
- added D505: 1N4148W, Diode_SMD:D_SOD-123, symbol Diode:1N4148W
- added K501: 9012, ADC_TEST:9012, symbol ADC_TEST:9012
- added Q502: BC847, Package_TO_SOT_SMD:SOT-23, symbol Transistor_BJT:BC847
- added Q503: MMBTA55, Package_TO_SOT_SMD:SOT-23, symbol ADC_TEST:MMBTA55
- added R523: 10k, Resistor_SMD:R_0603_1608Metric_Pad1.05x0.95mm_HandSolder, symbol Device:R
- added R524, R525: 4k7/.1%, Resistor_SMD:R_0603_1608Metric_Pad1.05x0.95mm_HandSolder, symbol Device:R
- added U513: LT1021-7, Package_SO:SOIC-8-N7_3.9x4.9mm_P1.27mm, symbol ADC_TEST:LT1021-7
Connections:
- net +18VF: now also R525.1
- net +5VF: now also D505.1 (K), K501.2
- net -14VF: now also Q503.3 (C), R524.2
- net AGNDF: now also U513.6 (Vout)
- net DGNDF: now also C525.1, Q502.2 (E)
- net at C506.1, R504.1, R505.1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: now also K501.4
- new net: D504.1 (K), R525.2, U513.2 (Vin)
- new net: D504.2 (A), Q503.1 (B), R524.1
- new net: K501.1, Q503.2 (E), U513.4 (GND)
- new net: D505.2 (A), K501.3, Q502.3 (C)
- new net: C525.2, Q502.1 (B), R523.1
- new net FPGA_AD_RFS_OPT: R523.2
Other:
- moved on the sheet: C506, C508, C509, C515, C517, C522, D501, D502, D503, Q501, R501, R502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

Commit message: PCB design
Parts:
- added R506, R508: 0, Resistor_SMD:R_0603_1608Metric_Pad1.05x0.95mm_HandSolder, symbol Device:R
- U504: renamed from U513; footprint Package_SO:SOIC-8-N7_3.9x4.9mm_P1.27mm -> Package_SO:SOIC-8_3.9x4.9mm_P1.27mm
- renumbered C525 to C501, C501 to C502, C502 to C503, C503 to C504, C504 to C505, C505 to C506, C510 to C508, C511 to C509, C512 to C510, C513 to C511, C506 to C512, C514 to C513, C516 to C514, C508 to C515, C509 to C516, C518 to C517, C519 to C518, C520 to C519, C521 to C520, C523 to C521, C515 to C522, C517 to C523, C522 to C525, D505 to D501, D504 to D502, D501 to D503, D502 to D504, D503 to D505, Q502 to Q501, Q503 to Q502, Q501 to Q503, R523 to R501, R524 to R502, R501 to R503, R525 to R504, R502 to R505, R503 to R507, R504 to R509, R505 to R510, R506 to R511, R507 to R512, R508 to R513, R509 to R514, R510 to R515, R511 to R516, R512 to R517, R513 to R518, R514 to R519, R515 to R520, R516 to R521, R517 to R522, R518 to R523, R519 to R524, R520 to R525, R521 to R526, R522 to R527, U504 to U505, U505 to U506, U506 to U507, U507 to U508, U508 to U509, U509 to U510, U510 to U511, U511 to U512, U512 to U513
Connections:
- net -14VF: now also R506.1
- net at R510.2, R515.2, U506.2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: now also K501.4, R508.1
- net at C512.1, R509.1, R510.1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: no longer K501.4
- net at D503.1 (K), Q503.3 (C), R507.1: now also R506.2
- net at K501.1, Q502.2 (E), U504.4 (GND): now also R508.2

Commit message: PCB design.
Parts:
- removed C509: 100n, Capacitor_SMD:C_0603_1608Metric_Pad1.05x0.95mm_HandSolder, symbol Device:C
- removed TP501, TP502, TP503: TestPoint, TestPoint:TestPoint_Loop_D2.60mm_Drill1.6mm_Beaded, symbol Connector:TestPoint
- renumbered C510 to C509, C511 to C510, C512 to C511, C513 to C512, C514 to C513, C515 to C514, C516 to C515, C517 to C516, C518 to C517, C519 to C518, C520 to C519, C521 to C520, C522 to C521, C523 to C522, C524 to C523, C525 to C524

Commit message: PCB design done.
Parts:
- R515: value 1k96/.1% -> 3k01/.1%
- R517: value 62k6/.1% -> 62k
- R520: value 400/.1% -> 0
Connections:
- net ADIN: now also U505.8; no longer U505.1
- net at U505.2: now also U505.1; no longer U505.8
- net +3.3VF renamed +3.3VP
- no-connect marks 8 -> 6
Other:
- note added: "Problem ???? Wrong value was selected."
Changed lines of the file:
@@
 	5600 1350 5700 1350
-Wire Wire Line
-	5600 850  5600 1350
 Wire Wire Line
 	6500 1200 6500 850
@@
 	0    1    1    0
 $EndComp
-Text HLabel 5350 1200 0    50   Input ~ 0
+Text HLabel 5600 850  0    50   Input ~ 0
 ADIN
-Wire Wire Line
-	5700 1200 5350 1200
 Wire Wire Line
 	6500 850  5600 850
@@
 P 10450 5600
 F 0 "R515" V 10243 5600 50  0000 C CNN
-F 1 "1k96/.1%" V 10334 5600 50  0000 C CNN
+F 1 "3k01/.1%" V 10334 5600 50  0000 C CNN
 F 2 "Resistor_SMD:R_0603_1608Metric_Pad1.05x0.95mm_HandSolder" V 10380 5600 50  0001 C CNN
 F 3 "~" H 10450 5600 50  0001 C CNN
@@
 	1    10450 7100
 	0    1    1    0
-$EndComp
-$Comp
-L ADC_TEST:OPA140 U?
-U 1 1 601E11FB
-P 9100 2300
-AR Path="/601E11FB" Ref="U?"  Part="1"
-AR Path="/5FCCC067/601E11FB" Ref="U509"  Part="1"
-F 0 "U509" H 9300 2550 50  0000 L CNN
-F 1 "OPA140" H 9200 2450 50  0000 L CNN
-F 2 "Package_SO:SOIC-8_3.9x4.9mm_P1.27mm" H 9150 2350 50  0001 C CNN
-F 3 "" H 9250 2450 50  0001 C CNN
-	1    9100 2300
-	1    0    0    -1
 $EndComp
 $Comp
@@
 Wire Wire Line
 	9000 1900 9000 1950
-NoConn ~ 9100 2600
-NoConn ~ 9200 2600
 $Comp
 L ADC_TEST:AGNDF #PWR?
@@
 AR Path="/602ADB44" Ref="U?"  Part="1"
 AR Path="/5FCCC067/602ADB44" Ref="U510"  Part="1"
-F 0 "U510" H 10600 6500 50  0000 L CNN
+F 0 "U510" H 10550 6500 50  0000 L CNN
 F 1 "OPA177" H 10500 6400 50  0000 L CNN
 F 2 "Package_SO:SOIC-8_3.9x4.9mm_P1.27mm" H 10450 6300 50  0001 C CNN
@@
 AR Path="/602EA97D" Ref="U?"  Part="1"
 AR Path="/5FCCC067/602EA97D" Ref="U508"  Part="1"
-F 0 "U508" H 8800 7000 50  0000 L CNN
+F 0 "U508" H 8750 7000 50  0000 L CNN
 F 1 "OPA177" H 8700 6900 50  0000 L CNN
 F 2 "Package_SO:SOIC-8_3.9x4.9mm_P1.27mm" H 8650 6800 50  0001 C CNN
@@
 AR Path="/60561E40" Ref="U?"  Part="1"
 AR Path="/5FCCC067/60561E40" Ref="U511"  Part="1"
-F 0 "U511" H 10850 2450 50  0000 L CNN
+F 0 "U511" H 10800 2450 50  0000 L CNN
 F 1 "OPA192" H 10750 2350 50  0000 L CNN
 F 2 "Package_SO:SOIC-8_3.9x4.9mm_P1.27mm" H 10700 2250 50  0001 C CNN
@@
 P 10500 4250
 F 0 "R517" V 10293 4250 50  0000 C CNN
-F 1 "62k6/.1%" V 10384 4250 50  0000 C CNN
+F 1 "62k" V 10384 4250 50  0000 C CNN
 F 2 "Resistor_SMD:R_0603_1608Metric_Pad1.05x0.95mm_HandSolder" V 10430 4250 50  0001 C CNN
 F 3 "~" H 10500 4250 50  0001 C CNN
@@
 AR Path="/6065D0D7" Ref="U?"  Part="1"
 AR Path="/5FCCC067/6065D0D7" Ref="U513"  Part="1"
-F 0 "U513" H 12750 2550 50  0000 L CNN
+F 0 "U513" H 12700 2550 50  0000 L CNN
 F 1 "LM311" H 12700 2450 50  0000 L CNN
 F 2 "Package_SO:SOIC-8_3.9x4.9mm_P1.27mm" H 12500 2300 50  0001 C CNN
@@
 Wire Wire Line
 	12400 3200 12400 2800
-$Comp
-L ADC_TEST:+3.3VF #PWR?
-U 1 1 606DD4C4
-P 12900 3200
-AR Path="/606DD4C4" Ref="#PWR?"  Part="1"
-AR Path="/5FCCC067/606DD4C4" Ref="#PWR0548"  Part="1"
-F 0 "#PWR0548" H 12900 3050 50  0001 C CNN
-F 1 "+3.3VF" V 12915 3328 50  0000 L CNN
-F 2 "" H 12900 3200 50  0001 C CNN
-F 3 "" H 12900 3200 50  0001 C CNN
-	1    12900 3200
-	0    1    1    0
-$EndComp
 Wire Wire Line
 	12900 3200 12850 3200
@@
 Wire Wire Line
 	13050 1800 13050 2300
-$Comp
-L ADC_TEST:+3.3VF #PWR?
-U 1 1 6073FFA9
-P 12500 1100
-AR Path="/6073FFA9" Ref="#PWR?"  Part="1"
-AR Path="/5FCCC067/6073FFA9" Ref="#PWR0546"  Part="1"
-F 0 "#PWR0546" H 12500 950 50  0001 C CNN
-F 1 "+3.3VF" H 12515 1273 50  0000 C CNN
-F 2 "" H 12500 1100 50  0001 C CNN
-F 3 "" H 12500 1100 50  0001 C CNN
-	1    12500 1100
-	1    0    0    -1
-$EndComp
-$Comp
-L ADC_TEST:+3.3VF #PWR?
-U 1 1 607403BE
-P 12200 1900
-AR Path="/607403BE" Ref="#PWR?"  Part="1"
-AR Path="/5FCCC067/607403BE" Ref="#PWR0544"  Part="1"
-F 0 "#PWR0544" H 12200 1750 50  0001 C CNN
-F 1 "+3.3VF" H 12215 2073 50  0000 C CNN
-F 2 "" H 12200 1900 50  0001 C CNN
-F 3 "" H 12200 1900 50  0001 C CNN
-	1    12200 1900
-	1    0    0    -1
-$EndComp
 Wire Wire Line
 	12200 1900 12200 1950
@@
 P 11050 4250
 F 0 "R520" V 10843 4250 50  0000 C CNN
-F 1 "400/.1%" V 10934 4250 50  0000 C CNN
+F 1 "0" V 10934 4250 50  0000 C CNN
 F 2 "Resistor_SMD:R_0603_1608Metric_Pad1.05x0.95mm_HandSolder" V 10980 4250 50  0001 C CNN
 F 3 "~" H 11050 4250 50  0001 C CNN
@@
 Connection ~ 7200 6150
 Connection ~ 6300 5400
+$Comp
+L power:+3.3VP #PWR0101
+U 1 1 5F88E174
+P 12200 1900
+F 0 "#PWR0101" H 12350 1850 50  0001 C CNN
+F 1 "+3.3VP" H 12215 2073 50  0000 C CNN
+F 2 "" H 12200 1900 50  0001 C CNN
+F 3 "" H 12200 1900 50  0001 C CNN
+	1    12200 1900
+	1    0    0    -1
+$EndComp
+$Comp
+L power:+3.3VP #PWR0102
+U 1 1 5F88E440
+P 12500 1100
+F 0 "#PWR0102" H 12650 1050 50  0001 C CNN
+F 1 "+3.3VP" H 12515 1273 50  0000 C CNN
+F 2 "" H 12500 1100 50  0001 C CNN
+F 3 "" H 12500 1100 50  0001 C CNN
+	1    12500 1100
+	1    0    0    -1
+$EndComp
+$Comp
+L power:+3.3VP #PWR0103
+U 1 1 5F891819
+P 12900 3200
+F 0 "#PWR0103" H 13050 3150 50  0001 C CNN
+F 1 "+3.3VP" V 12900 3350 50  0000 L CNN
+F 2 "" H 12900 3200 50  0001 C CNN
+F 3 "" H 12900 3200 50  0001 C CNN
+	1    12900 3200
+	0    1    1    0
+$EndComp
+$Comp
+L ADC_TEST:OPA140 U?
+U 1 1 601E11FB
+P 9100 2300
+AR Path="/601E11FB" Ref="U?"  Part="1"
+AR Path="/5FCCC067/601E11FB" Ref="U509"  Part="1"
+F 0 "U509" H 9250 2550 50  0000 L CNN
+F 1 "OPA140" H 9200 2450 50  0000 L CNN
+F 2 "Package_SO:SOIC-8_3.9x4.9mm_P1.27mm" H 9150 2350 50  0001 C CNN
+F 3 "" H 9250 2450 50  0001 C CNN
+	1    9100 2300
+	1    0    0    -1
+$EndComp
+Wire Wire Line
+	5700 1200 5600 1200
+Wire Wire Line
+	5600 1200 5600 1350
+Wire Wire Line
+	13050 2300 13650 2300
 Wire Wire Line
 	9450 2300 9450 3450
-Wire Wire Line
-	13050 2300 13650 2300
+Text Notes 11450 4250 0    50   ~ 0
+Problem ???? Wrong value was selected.
 $EndSCHEMATC
