File: hardware/project/ADC_Test/ADC_Test.sch (KiCad schematic (older format))
At the start: 3 parts, among them J101 RF_Shield_One_Piece, J102 Conn_01x02_Male, J103 Conn_01x04_Male

Commit message: Schematic design.
Other:
- note added: "1M - RS73F2BTTD1004B\n240k - RG2012N-244-W-T1\n22 - CPF1206B22RE1\n12k - ERA-3ARW123V\n39k - ERJ-P06F3902V\n93k - RK73H2ATTD9312D\n12k - RCS080512K0FKEA\n620 - RG2012N-621-W-T1 Only 2, for the rest standar values. \n4n7 - C1206C472FAGECTU\n62k6 - RN73H1JTTD6262B25\n400 - PAT0603E4000BST1\n3k9 - RG1608N-392-W-T1\n39k - ERA-3ARW393V\n62 - ERA-3AEB620V"
Changed lines of the file:
@@
 F0 "Power" 50
 F1 "Power.sch" 50
+F2 "FGPA_PWR_ON" I L 7600 5600 50
 $EndSheet
 $Sheet
@@
 Wire Wire Line
 	9250 4350 8950 4350
+Wire Wire Line
+	7600 800  7150 800
+Wire Wire Line
+	8950 900  9250 900
+Wire Wire Line
+	9250 800  8950 800
+Wire Wire Line
+	3450 1300 5050 1300
+Wire Wire Line
+	3450 1000 5050 1000
+Wire Wire Line
+	5050 900  3450 900
+Wire Wire Line
+	3450 800  5050 800
+Wire Wire Line
+	3450 1100 5050 1100
+Wire Wire Line
+	3450 1200 5050 1200
+Wire Wire Line
+	3450 1400 5050 1400
+$Sheet
+S 5050 700  2100 1750
+U 5FCCC067
+F0 "ADC" 50
+F1 "ADC.sch" 50
+F2 "FGPA_AD_IRN" I L 5050 900 50
+F3 "FGPA_AD_ID" I L 5050 1000 50
+F4 "FGPA_AD_IRP" I L 5050 1100 50
+F5 "FGPA_AD_IIN" I L 5050 1200 50
+F6 "ADIN" I R 7150 800 50
+F7 "AD_COMP" O L 5050 1300 50
+F8 "FPGA_AD_RFS" I L 5050 1400 50
+F9 "FPGA_SW_VRH" I L 5050 800 50
+F10 "VREF_-7V" O R 7150 900 50
+$EndSheet
+Wire Wire Line
+	7150 900  7600 900
+$Sheet
+S 7600 700  1350 2950
+U 601DD7F1
+F0 "Input" 50
+F1 "Input.sch" 50
+F2 "V_HIGH" I R 8950 800 50
+F3 "V_LOW" I R 8950 900 50
+F4 "ADIN" O L 7600 800 50
+F5 "VREF_-7V" I L 7600 900 50
+F6 "SR_CLK" I L 7600 3000 50
+F7 "SR_DAT" I L 7600 3100 50
+F8 "SR_LAT" I L 7600 3200 50
+$EndSheet
+Wire Wire Line
+	7150 5600 7600 5600
 $Sheet
 S 5050 2850 2100 3450
@@
 F19 "FPGA_SPI3_SCK" O L 5050 3950 50
 F20 "FPGA_UART2_CTRL_TTL" B L 5050 3700 50
-F21 "AMP_10MEG" O R 7150 3550 50
-F22 "RLY1_CTR" O R 7150 3450 50
-F23 "MCU_ADC1_AZ" O R 7150 3250 50
-F24 "MCU_ADC2_AZ" O R 7150 3150 50
-F25 "RLY2_CTR" O R 7150 3350 50
-$EndSheet
-$Sheet
-S 7600 700  1350 2950
-U 601DD7F1
-F0 "Input" 50
-F1 "Input.sch" 50
-F2 "AMP_10MEG" I L 7600 3550 50
-F3 "RLY1_CTR" I L 7600 3450 50
-F4 "MCU_ADC1_AZ" I L 7600 3250 50
-F5 "MCU_ADC2_AZ" I L 7600 3150 50
-F6 "RLY2_CTR" I L 7600 3350 50
-F7 "ADIN" O L 7600 800 50
-F8 "V_HIGH" I R 8950 800 50
-F9 "V_LOW" I R 8950 900 50
-$EndSheet
-Wire Wire Line
-	7600 3550 7150 3550
-Wire Wire Line
-	7600 3450 7150 3450
-Wire Wire Line
-	7600 3350 7150 3350
-Wire Wire Line
-	7600 3250 7150 3250
-Wire Wire Line
-	7600 3150 7150 3150
-Wire Wire Line
-	7600 800  7150 800
-Wire Wire Line
-	8950 900  9250 900
-Wire Wire Line
-	9250 800  8950 800
-Wire Wire Line
-	3450 1300 5050 1300
+F21 "FGPA_PWR_ON" O R 7150 5600 50
+F22 "SR_CLK" O R 7150 3000 50
+F23 "SR_DAT" O R 7150 3100 50
+F24 "SR_LAT" O R 7150 3200 50
+$EndSheet
+Wire Wire Line
+	7150 3200 7600 3200
+Wire Wire Line
+	7600 3100 7150 3100
+Wire Wire Line
+	7150 3000 7600 3000
 $Sheet
 S 1300 700  2150 5600
@@
 F10 "FPGA_SPI3_MISO" O R 3450 4050 50
 F11 "FPGA_SPI3_MOSI" I R 3450 4150 50
-F12 "FGPA_SW_VRH" O R 3450 800 50
-F13 "FGPA_AD_IRN" O R 3450 900 50
-F14 "FGPA_AD_IRP" O R 3450 1100 50
-F15 "FPGA_AD_IIN" O R 3450 1200 50
-F16 "FGPA_AD_ID" O R 3450 1000 50
+F12 "FGPA_AD_ID" O R 3450 1000 50
+F13 "FGPA_AD_VRH" O R 3450 800 50
+F14 "FGPA_AD_IRN" O R 3450 900 50
+F15 "FGPA_AD_IRP" O R 3450 1100 50
+F16 "FPGA_AD_IIN" O R 3450 1200 50
 F17 "FPGA_AD_RFS" O R 3450 1400 50
 $EndSheet
-Wire Wire Line
-	3450 1000 5050 1000
-Wire Wire Line
-	5050 900  3450 900
-Wire Wire Line
-	3450 800  5050 800
-Wire Wire Line
-	3450 1100 5050 1100
-Wire Wire Line
-	3450 1200 5050 1200
-Wire Wire Line
-	3450 1400 5050 1400
-$Sheet
-S 5050 700  2100 1750
-U 5FCCC067
-F0 "ADC" 50
-F1 "ADC.sch" 50
-F2 "FGPA_AD_IRN" I L 5050 900 50
-F3 "FGPA_AD_ID" I L 5050 1000 50
-F4 "FGPA_AD_IRP" I L 5050 1100 50
-F5 "FGPA_AD_IIN" I L 5050 1200 50
-F6 "ADIN" I R 7150 800 50
-F7 "AD_COMP" O L 5050 1300 50
-F8 "FPGA_AD_RFS" I L 5050 1400 50
-F9 "FPGA_SW_VRH" I L 5050 800 50
-F10 "VR_-7V" O R 7150 900 50
-$EndSheet
-Wire Wire Line
-	7150 900  7600 900
+Text Notes 4300 7600 0    50   ~ 0
+1M - RS73F2BTTD1004B\n240k - RG2012N-244-W-T1\n22 - CPF1206B22RE1\n12k - ERA-3ARW123V\n39k - ERJ-P06F3902V\n93k - RK73H2ATTD9312D\n12k - RCS080512K0FKEA\n620 - RG2012N-621-W-T1 Only 2, for the rest standar values. \n4n7 - C1206C472FAGECTU\n62k6 - RN73H1JTTD6262B25\n400 - PAT0603E4000BST1\n3k9 - RG1608N-392-W-T1\n39k - ERA-3ARW393V\n62 - ERA-3AEB620V
 $EndSCHEMATC

Commit message: Changes in documentation, schematics and PCB.
Changed lines of the file:
@@
 F9 "FPGA_SW_VRH" I L 5050 800 50
 F10 "VREF_-7V" O R 7150 900 50
+F11 "FPGA_AD_RFS_OPT" I L 5050 1500 50
 $EndSheet
 Wire Wire Line
@@
 F16 "FPGA_AD_IIN" O R 3450 1200 50
 F17 "FPGA_AD_RFS" O R 3450 1400 50
+F18 "FPGA_AD_RFS_OPT" O R 3450 1500 50
 $EndSheet
 Text Notes 4300 7600 0    50   ~ 0
 1M - RS73F2BTTD1004B\n240k - RG2012N-244-W-T1\n22 - CPF1206B22RE1\n12k - ERA-3ARW123V\n39k - ERJ-P06F3902V\n93k - RK73H2ATTD9312D\n12k - RCS080512K0FKEA\n620 - RG2012N-621-W-T1 Only 2, for the rest standar values. \n4n7 - C1206C472FAGECTU\n62k6 - RN73H1JTTD6262B25\n400 - PAT0603E4000BST1\n3k9 - RG1608N-392-W-T1\n39k - ERA-3ARW393V\n62 - ERA-3AEB620V
+Wire Wire Line
+	5050 1500 3450 1500
 $EndSCHEMATC

Commit message: PCB design
Parts:
- removed J101: RF_Shield_One_Piece, ADC_TEST:36107406S, symbol Device:RF_Shield_One_Piece
- removed J102: Conn_01x02_Male, Connector_PinHeader_2.54mm:PinHeader_1x02_P2.54mm_Vertical, symbol Connector:Conn_01x02_Male
- added J101: Conn_01x03_Male, Connector_PinHeader_2.54mm:PinHeader_1x03_P2.54mm_Vertical, symbol Connector:Conn_01x03_Male
- renumbered J103 to J102
Connections:
- net FPGA/FPGA_UART2_CTRL_TTL: now also J101.3 (Pin_3)
- net FPGA/FPGA_UART2_RX_TTL: now also J101.2 (Pin_2)
- net FPGA/FPGA_UART2_TX_TTL: now also J101.1 (Pin_1)
Changed lines of the file:
@@
 $EndSheet
 $Comp
-L Device:RF_Shield_One_Piece J101
-U 1 1 60B1EF8E
-P 2450 7000
-F 0 "J101" H 3080 6989 50  0000 L CNN
-F 1 "RF_Shield_One_Piece" H 3080 6898 50  0000 L CNN
-F 2 "ADC_TEST:36107406S" H 2450 6900 50  0001 C CNN
-F 3 "~" H 2450 6900 50  0001 C CNN
-	1    2450 7000
-	1    0    0    -1
-$EndComp
-$Comp
-L ADC_TEST:AGNDF #PWR0101
-U 1 1 60B1FAB2
-P 2450 7400
-F 0 "#PWR0101" H 2450 7150 50  0001 C CNN
-F 1 "AGNDF" H 2455 7227 50  0000 C CNN
-F 2 "" H 2450 7400 50  0001 C CNN
-F 3 "" H 2450 7400 50  0001 C CNN
-	1    2450 7400
-	1    0    0    -1
-$EndComp
-$Comp
-L Connector:Conn_01x04_Male J103
+L Connector:Conn_01x04_Male J102
 U 1 1 5FF3F385
 P 3800 4700
-F 0 "J103" H 3908 4981 50  0000 C CNN
+F 0 "J102" H 3908 4981 50  0000 C CNN
 F 1 "Conn_01x04_Male" H 3908 4890 50  0000 C CNN
 F 2 "Connector_PinHeader_2.54mm:PinHeader_1x04_P2.54mm_Vertical" H 3800 4700 50  0001 C CNN
@@
 Wire Wire Line
 	3450 3350 5050 3350
-$Comp
-L Connector:Conn_01x02_Male J102
-U 1 1 5FF42F37
-P 3800 2950
-F 0 "J102" H 3908 3131 50  0000 C CNN
-F 1 "Conn_01x02_Male" H 3908 3040 50  0000 C CNN
-F 2 "Connector_PinHeader_2.54mm:PinHeader_1x02_P2.54mm_Vertical" H 3800 2950 50  0001 C CNN
-F 3 "~" H 3800 2950 50  0001 C CNN
-	1    3800 2950
-	1    0    0    -1
-$EndComp
-Wire Wire Line
-	3450 3500 4300 3500
-Wire Wire Line
-	4300 3500 4300 3050
-Wire Wire Line
-	4300 3050 4000 3050
-Wire Wire Line
-	3450 3600 4400 3600
-Wire Wire Line
-	4400 3600 4400 2950
-Wire Wire Line
-	4400 2950 4000 2950
-Wire Wire Line
-	4300 3500 5050 3500
-Connection ~ 4300 3500
-Wire Wire Line
-	4400 3600 5050 3600
-Connection ~ 4400 3600
-Wire Wire Line
-	3450 3700 5050 3700
+Wire Wire Line
+	4300 2900 4000 2900
+Wire Wire Line
+	4400 2800 4000 2800
+Wire Wire Line
+	3450 3700 4150 3700
 Wire Wire Line
 	7150 4000 7600 4000
@@
 Wire Wire Line
 	5050 1500 3450 1500
+$Comp
+L Connector:Conn_01x03_Male J101
+U 1 1 5FF53AC2
+P 3800 2900
+F 0 "J101" H 3908 3181 50  0000 C CNN
+F 1 "Conn_01x03_Male" H 3908 3090 50  0000 C CNN
+F 2 "Connector_PinHeader_2.54mm:PinHeader_1x03_P2.54mm_Vertical" H 3800 2900 50  0001 C CNN
+F 3 "~" H 3800 2900 50  0001 C CNN
+	1    3800 2900
+	1    0    0    -1
+$EndComp
+Wire Wire Line
+	4150 3700 4150 3000
+Wire Wire Line
+	4150 3000 4000 3000
+Connection ~ 4150 3700
+Wire Wire Line
+	4150 3700 5050 3700
+Wire Wire Line
+	3450 3600 4300 3600
+Wire Wire Line
+	3450 3500 4400 3500
+Wire Wire Line
+	4300 2900 4300 3600
+Connection ~ 4300 3600
+Wire Wire Line
+	4300 3600 5050 3600
+Wire Wire Line
+	4400 2800 4400 3500
+Connection ~ 4400 3500
+Wire Wire Line
+	4400 3500 5050 3500
 $EndSCHEMATC

Commit message: PCB design.
Other:
- moved on the sheet: J101
Changed lines of the file:
@@
 	3450 3350 5050 3350
 Wire Wire Line
-	4300 2900 4000 2900
+	4300 2800 4000 2800
 Wire Wire Line
-	4400 2800 4000 2800
+	4400 2700 4000 2700
 Wire Wire Line
 	3450 3700 4150 3700
@@
 F10 "REF_CLK" B R 7150 4900 50
 F11 "NRST" B R 7150 4800 50
-F12 "FPGA_IO1" B L 5050 3250 50
-F13 "FPGA_IO2" B L 5050 3350 50
+F12 "FPGA_IO1" B L 5050 3050 50
+F13 "FPGA_IO2" B L 5050 3150 50
 F14 "FPGA_UART2_RX_TTL" B L 5050 3600 50
 F15 "FPGA_UART2_TX_TTL" B L 5050 3500 50
@@
 F23 "SR_DAT" O R 7150 3100 50
 F24 "SR_LAT" O R 7150 3200 50
+F25 "FPGA_IO3" B L 5050 3250 50
+F26 "FPGA_IO4" B L 5050 3350 50
 $EndSheet
 Wire Wire Line
@@
 F1 "FPGA.sch" 50
 F2 "ADC_COMP" I R 3450 1300 50
-F3 "FPGA_IO1" B R 3450 3250 50
-F4 "FPGA_IO2" B R 3450 3350 50
+F3 "FPGA_IO1" B R 3450 3050 50
+F4 "FPGA_IO2" B R 3450 3150 50
 F5 "FPGA_UART2_TX_TTL" B R 3450 3500 50
 F6 "FPGA_UART2_RX_TTL" B R 3450 3600 50
@@
 F17 "FPGA_AD_RFS" O R 3450 1400 50
 F18 "FPGA_AD_RFS_OPT" O R 3450 1500 50
+F19 "FPGA_IO3" B R 3450 3250 50
+F20 "FPGA_IO4" B R 3450 3350 50
 $EndSheet
 Text Notes 4300 7600 0    50   ~ 0
@@
 L Connector:Conn_01x03_Male J101
 U 1 1 5FF53AC2
-P 3800 2900
-F 0 "J101" H 3908 3181 50  0000 C CNN
-F 1 "Conn_01x03_Male" H 3908 3090 50  0000 C CNN
-F 2 "Connector_PinHeader_2.54mm:PinHeader_1x03_P2.54mm_Vertical" H 3800 2900 50  0001 C CNN
-F 3 "~" H 3800 2900 50  0001 C CNN
-	1    3800 2900
+P 3800 2800
+F 0 "J101" H 3908 3081 50  0000 C CNN
+F 1 "Conn_01x03_Male" H 3908 2990 50  0000 C CNN
+F 2 "Connector_PinHeader_2.54mm:PinHeader_1x03_P2.54mm_Vertical" H 3800 2800 50  0001 C CNN
+F 3 "~" H 3800 2800 50  0001 C CNN
+	1    3800 2800
 	1    0    0    -1
 $EndComp
 Wire Wire Line
-	4150 3700 4150 3000
+	4150 3700 4150 2900
 Wire Wire Line
-	4150 3000 4000 3000
+	4150 2900 4000 2900
 Connection ~ 4150 3700
 Wire Wire Line
@@
 	3450 3500 4400 3500
 Wire Wire Line
-	4300 2900 4300 3600
+	4300 2800 4300 3600
 Connection ~ 4300 3600
 Wire Wire Line
 	4300 3600 5050 3600
 Wire Wire Line
-	4400 2800 4400 3500
+	4400 2700 4400 3500
 Connection ~ 4400 3500
 Wire Wire Line
 	4400 3500 5050 3500
+Wire Wire Line
+	3450 3050 5050 3050
+Wire Wire Line
+	3450 3150 5050 3150
 $EndSCHEMATC

Commit message: PCB design done.
Changed lines of the file:
@@
 F0 "Power" 50
 F1 "Power.sch" 50
-F2 "FGPA_PWR_ON" I L 7600 5600 50
 $EndSheet
 $Sheet
@@
 F8 "SR_LAT" I L 7600 3200 50
 $EndSheet
-Wire Wire Line
-	7150 5600 7600 5600
 $Sheet
 S 5050 2850 2100 3450
@@
 F19 "FPGA_SPI3_SCK" O L 5050 3950 50
 F20 "FPGA_UART2_CTRL_TTL" B L 5050 3700 50
-F21 "FGPA_PWR_ON" O R 7150 5600 50
-F22 "SR_CLK" O R 7150 3000 50
-F23 "SR_DAT" O R 7150 3100 50
-F24 "SR_LAT" O R 7150 3200 50
-F25 "FPGA_IO3" B L 5050 3250 50
-F26 "FPGA_IO4" B L 5050 3350 50
-$EndSheet
-Wire Wire Line
+F21 "SR_CLK" O R 7150 3000 50
+F22 "SR_DAT" O R 7150 3100 50
+F23 "SR_LAT" O R 7150 3200 50
+F24 "FPGA_IO3" B L 5050 3250 50
+F25 "FPGA_IO4" B L 5050 3350 50
+$EndSheet
+Wire Wire Line
