File: hardware/project/ADC_Test/MCU.sch (KiCad schematic (older format))
At the start: 36 parts, among them J201 Conn_02x01, J202 20021111-00010T4LF, U201 STM32H743ZI/STM32F765ZGT6, Y201 NX3225GD-8MHZ-STD-CRA-3

Commit message: Schematic design.
Parts:
- removed C203: 100n, Capacitor_SMD:C_0603_1608Metric_Pad1.05x0.95mm_HandSolder, symbol Device:C
- added R705, R706: 4k7, Resistor_SMD:R_0603_1608Metric_Pad1.05x0.95mm_HandSolder, symbol Device:R
- added U702: 24LC08B-E/MS, Package_SO:MSOP-8_3x3mm_P0.65mm, symbol Memory_EEPROM:24LC08
- renumbered C201 to C701, C202 to C702, C204 to C703, C205 to C704, C206 to C705, C207 to C706, C208 to C707, C209 to C708, C210 to C709, C211 to C710, C212 to C711, C213 to C712, C214 to C713, C215 to C714, C216 to C715, C217 to C716, C218 to C717, C219 to C718, C220 to C719, C221 to C720, C222 to C721, D201 to D701, D202 to D702, D203 to D703, FB201 to FB701, J201 to J701, J202 to J702, R201 to R701, R202 to R702, R203 to R703, R204 to R704, R205 to R707, R206 to R708, U201 to U701, Y201 to Y701
Connections:
- net +3.3VF: now also R705.1, R706.1, U702.8 (VCC)
- net SR_LAT: now reaches U701.1 (PE2,TRACECLK,SPI4_SCK,SAI1_MCLK_A,QUADSPI_BK1_IO2,ETH_MII_TXD3,FMC_A23,EVENTOUT)
- net SR_DAT: now reaches U701.2 (PE3,TRACED0,SAI1_SD_B,FMC_A19,EVENTOUT)
- net SR_CLK: now reaches U701.3 (PE4,TRACED1,SPI4_NSS,SAI1_FS_A,DFSDM1_DATIN3,FMC_A20,DCMI_D4,LCD_B0,EVENTOUT)
- net FGPA_PWR_ON: now reaches U701.68 (PE15,TIM1_BKIN,FMC_D12,LCD_R7,EVENTOUT)
- net EEPROM_WP: now reaches U701.80 (PD11,I2C4_SMBA,USART3_CTS,QUADSPI_BK1_IO0,SAI2_SD_A,FMC_A16,FMC_CLE,EVENTOUT)
- net EEPROM_WP: now also U702.7 (WP)
- net EEPROM_SCL: now reaches U701.81 (PD12,TIM4_CH1,LPTIM1_IN1,I2C4_SCL,USART3_RTS,QUADSPI_BK1_IO1,SAI2_FS_A,FMC_A17,FMC_ALE,EVENTOUT)
- net EEPROM_SCL: now also R706.2, U702.6 (SCL)
- net EEPROM_SDA: now reaches U701.82 (PD13,TIM4_CH2,LPTIM1_OUT,I2C4_SDA,QUADSPI_BK1_IO3,SAI2_SCK_A,FMC_A18,EVENTOUT)
- net EEPROM_SDA: now also R705.2, U702.5 (SDA)
- net AMP_10MEG: no longer names the net of U701.87 (PG2,FMC_A12,EVENTOUT)
- net DGNDF renamed GND
- net GND: now also U702.1 (A0), U702.2 (A1), U702.3 (A2), U702.4 (GND)
- net MCU_ADC1_AZ: no longer names the net of U701.56 (PG0,FMC_A10,EVENTOUT)
- net MCU_ADC2_AZ: no longer names the net of U701.57 (PG1,FMC_A11,EVENTOUT)
- net RLY1_CTR: no longer names the net of U701.89 (PG4,FMC_A14,FMC_BA0,EVENTOUT)
- net RLY2_CTR: no longer names the net of U701.88 (PG3,FMC_A13,EVENTOUT)
- no-connect marks 87 -> 85
Other:
- moved on the sheet: J702

Commit message: PCB design
Parts:
- removed J701: Conn_02x01, Connector_PinHeader_2.54mm:PinHeader_1x02_P2.54mm_Vertical, symbol Connector_Generic:Conn_02x01
- removed R701: 10k, Resistor_SMD:R_0603_1608Metric_Pad1.05x0.95mm_HandSolder, symbol Device:R
- renumbered J702 to J701, R702 to R701, R703 to R702, R704 to R703, R705 to R704, R706 to R705, R707 to R706, R708 to R707
Connections:
- net MCU_DEFAULT: no longer names the net of U701.34 (PA0,TIM2_CH1,TIM2_ETR,TIM5_CH1,TIM8_ETR,USART2_CTS,UART4_TX,SAI2_SD_B,ETH_MII_CRS,EVENTOUT,ADC1_IN0,ADC2_IN0,ADC3_IN0,WKUP1)
- no-connect marks 85 -> 86
Changed lines of the file:
@@
 	8850 9050 8850 9100
 $Comp
-L power:GND #PWR0717
+L power:GND #PWR0715
 U 1 1 5DAA3278
 P 8850 9100
-F 0 "#PWR0717" H 8850 8850 50  0001 C CNN
+F 0 "#PWR0715" H 8850 8850 50  0001 C CNN
 F 1 "GND" H 8855 8927 50  0000 C CNN
 F 2 "" H 8850 9100 50  0001 C CNN
@@
 $EndComp
 $Comp
-L Device:R R707
+L Device:R R706
 U 1 1 5DAA6CE1
 P 14600 8900
-F 0 "R707" H 14670 8946 50  0000 L CNN
+F 0 "R706" H 14670 8946 50  0000 L CNN
 F 1 "10k" H 14670 8855 50  0000 L CNN
 F 2 "Resistor_SMD:R_0603_1608Metric_Pad1.05x0.95mm_HandSolder" V 14530 8900 50  0001 C CNN
@@
 	14600 8700 14550 8700
 $Comp
-L Device:R R708
+L Device:R R707
 U 1 1 5DAA8BD1
 P 15200 8100
-F 0 "R708" H 15270 8146 50  0000 L CNN
+F 0 "R707" H 15270 8146 50  0000 L CNN
 F 1 "10k" H 15270 8055 50  0000 L CNN
 F 2 "Resistor_SMD:R_0603_1608Metric_Pad1.05x0.95mm_HandSolder" V 15130 8100 50  0001 C CNN
@@
 Connection ~ 15200 8300
 $Comp
-L power:GND #PWR0723
+L power:GND #PWR0721
 U 1 1 5DAAC0BD
 P 15200 8650
-F 0 "#PWR0723" H 15200 8400 50  0001 C CNN
+F 0 "#PWR0721" H 15200 8400 50  0001 C CNN
 F 1 "GND" H 15205 8477 50  0000 C CNN
 F 2 "" H 15200 8650 50  0001 C CNN
@@
 $EndComp
 $Comp
-L power:GND #PWR0721
+L power:GND #PWR0719
 U 1 1 5DAACD0D
 P 14600 9050
-F 0 "#PWR0721" H 14600 8800 50  0001 C CNN
+F 0 "#PWR0719" H 14600 8800 50  0001 C CNN
 F 1 "GND" H 14605 8877 50  0000 C CNN
 F 2 "" H 14600 9050 50  0001 C CNN
@@
 Connection ~ 3100 8300
 $Comp
-L Connector_Generic:Conn_02x05_Odd_Even J702
+L Connector_Generic:Conn_02x05_Odd_Even J701
 U 1 1 5DA8679B
 P 8200 10450
-F 0 "J702" H 8250 10867 50  0000 C CNN
+F 0 "J701" H 8250 10867 50  0000 C CNN
 F 1 "20021111-00010T4LF" H 8250 10776 50  0000 C CNN
 F 2 "Connector_PinHeader_1.27mm:PinHeader_2x05_P1.27mm_Vertical" H 8200 10450 50  0001 C CNN
@@
 	7750 10350 8000 10350
 $Comp
-L power:GND #PWR0715
+L power:GND #PWR0713
 U 1 1 5DAA5490
 P 7750 10700
-F 0 "#PWR0715" H 7750 10450 50  0001 C CNN
+F 0 "#PWR0713" H 7750 10450 50  0001 C CNN
 F 1 "GND" H 7755 10527 50  0000 C CNN
 F 2 "" H 7750 10700 50  0001 C CNN
@@
 MCU_VDDA
 $Comp
-L power:GND #PWR0709
+L power:GND #PWR0707
 U 1 1 5DACCD5C
 P 3100 8500
-F 0 "#PWR0709" H 3100 8250 50  0001 C CNN
+F 0 "#PWR0707" H 3100 8250 50  0001 C CNN
 F 1 "GND" V 3105 8372 50  0000 R CNN
 F 2 "" H 3100 8500 50  0001 C CNN
@@
 	3100 8700 3150 8700
 $Comp
-L power:GND #PWR0710
+L power:GND #PWR0708
 U 1 1 5DAD7BE9
 P 3100 9100
-F 0 "#PWR0710" H 3100 8850 50  0001 C CNN
+F 0 "#PWR0708" H 3100 8850 50  0001 C CNN
 F 1 "GND" H 3105 8927 50  0000 C CNN
 F 2 "" H 3100 9100 50  0001 C CNN
@@
 	1150 10900 1650 10900
 $Comp
-L power:GND #PWR0712
+L power:GND #PWR0710
 U 1 1 5DB438B1
 P 3650 10950
-F 0 "#PWR0712" H 3650 10700 50  0001 C CNN
+F 0 "#PWR0710" H 3650 10700 50  0001 C CNN
 F 1 "GND" H 3655 10777 50  0000 C CNN
 F 2 "" H 3650 10950 50  0001 C CNN
@@
 	7100 10500 7100 10550
 $Comp
-L power:GND #PWR0713
+L power:GND #PWR0711
 U 1 1 5DB72CF5
 P 7100 10950
-F 0 "#PWR0713" H 7100 10700 50  0001 C CNN
+F 0 "#PWR0711" H 7100 10700 50  0001 C CNN
 F 1 "GND" H 7105 10777 50  0000 C CNN
 F 2 "" H 7100 10950 50  0001 C CNN
@@
 Text Label 7600 10500 2    50   ~ 0
 MCU_VDDA
-$Comp
-L Connector_Generic:Conn_02x01 J701
-U 1 1 5DB87F87
-P 650 8700
-F 0 "J701" V 654 8780 50  0000 L CNN
-F 1 "Conn_02x01" V 745 8780 50  0000 L CNN
-F 2 "Connector_PinHeader_2.54mm:PinHeader_1x02_P2.54mm_Vertical" H 650 8700 50  0001 C CNN
-F 3 "~" H 650 8700 50  0001 C CNN
-	1    650  8700
-	0    1    1    0
-$EndComp
-$Comp
-L power:GND #PWR0702
-U 1 1 5DB88AAB
-P 650 9000
-F 0 "#PWR0702" H 650 8750 50  0001 C CNN
-F 1 "GND" H 655 8827 50  0000 C CNN
-F 2 "" H 650 9000 50  0001 C CNN
-F 3 "" H 650 9000 50  0001 C CNN
-	1    650  9000
-	1    0    0    -1
-$EndComp
-$Comp
-L Device:R R701
-U 1 1 5DB8FF79
-P 650 8250
-F 0 "R701" H 580 8204 50  0000 R CNN
-F 1 "10k" H 580 8295 50  0000 R CNN
-F 2 "Resistor_SMD:R_0603_1608Metric_Pad1.05x0.95mm_HandSolder" V 580 8250 50  0001 C CNN
-F 3 "~" H 650 8250 50  0001 C CNN
-	1    650  8250
-	-1   0    0    1
-$EndComp
-Wire Wire Line
-	650  8500 650  8450
-Wire Wire Line
-	650  8450 1200 8450
-Connection ~ 650  8450
-Wire Wire Line
-	650  8450 650  8400
-Text Label 1200 8450 2    50   ~ 0
-MCU_DEFAULT
 $Comp
 L Device:C C709
@@
 	1950 7700 1950 7950
 $Comp
-L power:GND #PWR0707
+L power:GND #PWR0705
 U 1 1 5DBC271D
 P 2200 8350
-F 0 "#PWR0707" H 2200 8100 50  0001 C CNN
+F 0 "#PWR0705" H 2200 8100 50  0001 C CNN
 F 1 "GND" H 2205 8177 50  0000 C CNN
 F 2 "" H 2200 8350 50  0001 C CNN
@@
 	1750 1700 1750 1650
 $Comp
-L power:GND #PWR0705
+L power:GND #PWR0703
 U 1 1 5DC11C96
 P 1500 1750
-F 0 "#PWR0705" H 1500 1500 50  0001 C CNN
+F 0 "#PWR0703" H 1500 1500 50  0001 C CNN
 F 1 "GND" H 1505 1577 50  0000 C CNN
 F 2 "" H 1500 1750 50  0001 C CNN
@@
 Wire Wire Line
 	3650 10900 4150 10900
-Wire Wire Line
-	3150 3200 2600 3200
-Text Label 2600 3200 0    50   ~ 0
-MCU_DEFAULT
 Connection ~ 6650 10500
 Wire Wire Line
@@
 Connection ~ 7100 10500
 $Comp
-L Device:R R702
+L Device:R R701
 U 1 1 5E648C3B
 P 2750 6550
-F 0 "R702" V 2543 6550 50  0000 C CNN
+F 0 "R701" V 2543 6550 50  0000 C CNN
 F 1 "680" V 2634 6550 50  0000 C CNN
 F 2 "Resistor_SMD:R_0603_1608Metric_Pad1.05x0.95mm_HandSolder" V 2680 6550 50  0001 C CNN
@@
 $EndComp
 $Comp
-L Device:R R703
+L Device:R R702
 U 1 1 5E64A32E
 P 2750 6950
-F 0 "R703" V 2543 6950 50  0000 C CNN
+F 0 "R702" V 2543 6950 50  0000 C CNN
 F 1 "560" V 2634 6950 50  0000 C CNN
 F 2 "Resistor_SMD:R_0603_1608Metric_Pad1.05x0.95mm_HandSolder" V 2680 6950 50  0001 C CNN
@@
 $EndComp
 $Comp
-L Device:R R704
+L Device:R R703
 U 1 1 5E64A698
 P 2750 7350
-F 0 "R704" V 2543 7350 50  0000 C CNN
+F 0 "R703" V 2543 7350 50  0000 C CNN
 F 1 "680" V 2634 7350 50  0000 C CNN
 F 2 "Resistor_SMD:R_0603_1608Metric_Pad1.05x0.95mm_HandSolder" V 2680 7350 50  0001 C CNN
@@
 	2150 6950 2200 6950
 $Comp
-L ADC_TEST:+3.3VF #PWR0716
+L ADC_TEST:+3.3VF #PWR0714
 U 1 1 5E419507
 P 8850 800
-F 0 "#PWR0716" H 8850 650 50  0001 C CNN
+F 0 "#PWR0714" H 8850 650 50  0001 C CNN
 F 1 "+3.3VF" H 8865 973 50  0000 C CNN
 F 2 "" H 8850 800 50  0001 C CNN
@@
 $EndComp
 $Comp
-L ADC_TEST:+3.3VF #PWR0711
+L ADC_TEST:+3.3VF #PWR0709
 U 1 1 5E4217A1
 P 3650 10450
-F 0 "#PWR0711" H 3650 10300 50  0001 C CNN
+F 0 "#PWR0709" H 3650 10300 50  0001 C CNN
 F 1 "+3.3VF" H 3665 10623 50  0000 C CNN
 F 2 "" H 3650 10450 50  0001 C CNN
@@
 $EndComp
 $Comp
-L ADC_TEST:+3.3VF #PWR0701
-U 1 1 5E422513
-P 650 8100
-F 0 "#PWR0701" H 650 7950 50  0001 C CNN
-F 1 "+3.3VF" H 665 8273 50  0000 C CNN
-F 2 "" H 650 8100 50  0001 C CNN
-F 3 "" H 650 8100 50  0001 C CNN
-	1    650  8100
-	1    0    0    -1
-$EndComp
-$Comp
-L ADC_TEST:+3.3VF #PWR0714
+L ADC_TEST:+3.3VF #PWR0712
 U 1 1 5E423A04
 P 7750 10150
-F 0 "#PWR0714" H 7750 10000 50  0001 C CNN
+F 0 "#PWR0712" H 7750 10000 50  0001 C CNN
 F 1 "+3.3VF" H 7765 10323 50  0000 C CNN
 F 2 "" H 7750 10150 50  0001 C CNN
@@
 $EndComp
 $Comp
-L ADC_TEST:+3.3VF #PWR0722
+L ADC_TEST:+3.3VF #PWR0720
 U 1 1 5E426FFF
 P 15200 7950
-F 0 "#PWR0722" H 15200 7800 50  0001 C CNN
+F 0 "#PWR0720" H 15200 7800 50  0001 C CNN
 F 1 "+3.3VF" H 15215 8123 50  0000 C CNN
 F 2 "" H 15200 7950 50  0001 C CNN
@@
 $EndComp
 $Comp
-L ADC_TEST:+3.3VF #PWR0708
+L ADC_TEST:+3.3VF #PWR0706
 U 1 1 5E4281F0
 P 3050 8700
-F 0 "#PWR0708" H 3050 8550 50  0001 C CNN
+F 0 "#PWR0706" H 3050 8550 50  0001 C CNN
 F 1 "+3.3VF" V 3050 8850 50  0000 L CNN
 F 2 "" H 3050 8700 50  0001 C CNN
@@
 $EndComp
 $Comp
-L ADC_TEST:+3.3VF #PWR0706
+L ADC_TEST:+3.3VF #PWR0704
 U 1 1 5E42C5D5
 P 2150 6950
-F 0 "#PWR0706" H 2150 6800 50  0001 C CNN
+F 0 "#PWR0704" H 2150 6800 50  0001 C CNN
 F 1 "+3.3VF" V 2150 7100 50  0000 L CNN
 F 2 "" H 2150 6950 50  0001 C CNN
@@
 NoConn ~ 14550 6600
 $Comp
-L ADC_TEST:+3.3VF #PWR0703
+L ADC_TEST:+3.3VF #PWR0701
 U 1 1 5E41DE54
 P 650 9600
-F 0 "#PWR0703" H 650 9450 50  0001 C CNN
+F 0 "#PWR0701" H 650 9450 50  0001 C CNN
 F 1 "+3.3VF" H 665 9773 50  0000 C CNN
 F 2 "" H 650 9600 50  0001 C CNN
@@
 	650  10100 650  10000
 $Comp
-L power:GND #PWR0704
+L power:GND #PWR0702
 U 1 1 5E1764D7
 P 650 10100
-F 0 "#PWR0704" H 650 9850 50  0001 C CNN
+F 0 "#PWR0702" H 650 9850 50  0001 C CNN
 F 1 "GND" H 655 9927 50  0000 C CNN
 F 2 "" H 650 10100 50  0001 C CNN
@@
 	9400 10350 9400 10250
 $Comp
-L power:GND #PWR0719
+L power:GND #PWR0717
 U 1 1 602F689C
 P 9850 10750
-F 0 "#PWR0719" H 9850 10500 50  0001 C CNN
+F 0 "#PWR0717" H 9850 10500 50  0001 C CNN
 F 1 "GND" H 9855 10577 50  0000 C CNN
 F 2 "" H 9850 10750 50  0001 C CNN
@@
 EEPROM_SDA
 $Comp
-L ADC_TEST:+3.3VF #PWR0718
+L ADC_TEST:+3.3VF #PWR0716
 U 1 1 60371547
 P 9850 10050
-F 0 "#PWR0718" H 9850 9900 50  0001 C CNN
+F 0 "#PWR0716" H 9850 9900 50  0001 C CNN
 F 1 "+3.3VF" H 9865 10223 50  0000 C CNN
 F 2 "" H 9850 10050 50  0001 C CNN
@@
 $EndComp
 $Comp
-L Device:R R705
+L Device:R R704
 U 1 1 60399835
 P 11000 10050
-F 0 "R705" H 11070 10096 50  0000 L CNN
+F 0 "R704" H 11070 10096 50  0000 L CNN
 F 1 "4k7" H 11070 10005 50  0000 L CNN
 F 2 "Resistor_SMD:R_0603_1608Metric_Pad1.05x0.95mm_HandSolder" V 10930 10050 50  0001 C CNN
@@
 	14550 4200 15100 4200
 $Comp
-L Device:R R706
+L Device:R R705
 U 1 1 603C8474
 P 11400 10050
-F 0 "R706" H 11470 10096 50  0000 L CNN
+F 0 "R705" H 11470 10096 50  0000 L CNN
 F 1 "4k7" H 11470 10005 50  0000 L CNN
 F 2 "Resistor_SMD:R_0603_1608Metric_Pad1.05x0.95mm_HandSolder" V 11330 10050 50  0001 C CNN
@@
 	11400 9850 11400 9900
 $Comp
-L ADC_TEST:+3.3VF #PWR0720
+L ADC_TEST:+3.3VF #PWR0718
 U 1 1 603F2C8A
 P 11200 9800
-F 0 "#PWR0720" H 11200 9650 50  0001 C CNN
+F 0 "#PWR0718" H 11200 9650 50  0001 C CNN
 F 1 "+3.3VF" H 11215 9973 50  0000 C CNN
 F 2 "" H 11200 9800 50  0001 C CNN
@@
 NoConn ~ 14550 4300
 NoConn ~ 14550 4400
+NoConn ~ 3150 3200
 $EndSCHEMATC

Commit message: PCB design.
Parts:
- renumbered R704 to R701, R705 to R702, R706 to R703, R701 to R704, R702 to R705, R703 to R706
Connections:
- net SR_CLK: now also U701.86 (PD15,TIM4_CH4,UART8_RTS,FMC_D1,EVENTOUT); no longer U701.3 (PE4,TRACED1,SPI4_NSS,SAI1_FS_A,DFSDM1_DATIN3,FMC_A20,DCMI_D4,LCD_B0,EVENTOUT)
- net SR_DAT: now also U701.92 (PG7,SAI1_MCLK_A,USART6_CK,FMC_INT,DCMI_D13,LCD_CLK,EVENTOUT); no longer U701.2 (PE3,TRACED0,SAI1_SD_B,FMC_A19,EVENTOUT)
- net SR_LAT: now also U701.76 (PB15,RTC_REFIN,TIM1_CH3N,TIM8_CH3N,USART1_RX,SPI2_MOSI,I2S2_SD,DFSDM1_CKIN2,UART4_CTS,TIM12_CH2,SDMMC2_D1,OTG_HS_DP,EVENTOUT); no longer U701.1 (PE2,TRACECLK,SPI4_SCK,SAI1_MCLK_A,QUADSPI_BK1_IO2,ETH_MII_TXD3,FMC_A23,EVENTOUT)
- net FPGA_IO3: now reaches U701.115 (PD1,DFSDM1_DATIN6,DFSDM1_CKIN7,UART4_TX,CAN1_TX,FMC_D3,EVENTOUT)
- net FPGA_IO4: now reaches U701.116 (PD2,TRACED2,TIM3_ETR,UART5_RX,SDMMC1_CMD,DCMI_D11,EVENTOUT)
- net at R704.1: now also U701.1 (PE2,TRACECLK,SPI4_SCK,SAI1_MCLK_A,QUADSPI_BK1_IO2,ETH_MII_TXD3,FMC_A23,EVENTOUT); no longer U701.7 (PC13,EVENTOUT,RTC_TAMP2,RTC_TS,WKUP5)
- net at R705.1: now also U701.2 (PE3,TRACED0,SAI1_SD_B,FMC_A19,EVENTOUT); no longer U701.8 (PC14,EVENTOUT,OSC32_IN)
- net at R706.1: now also U701.3 (PE4,TRACED1,SPI4_NSS,SAI1_FS_A,DFSDM1_DATIN3,FMC_A20,DCMI_D4,LCD_B0,EVENTOUT); no longer U701.9 (PC15,EVENTOUT,OSC32_OUT)
- no-connect marks 86 -> 84
Other:
- moved on the sheet: D701, D702, D703, R704, R705, R706

Commit message: PCB design done.
Connections:
- net FGPA_PWR_ON: no longer names the net of U701.68 (PE15,TIM1_BKIN,FMC_D12,LCD_R7,EVENTOUT)
- no-connect marks 84 -> 85
Changed lines of the file:
@@
 NoConn ~ 14550 1500
 NoConn ~ 14550 1600
-Text HLabel 14600 6100 2    50   Output ~ 0
-FGPA_PWR_ON
-Wire Wire Line
-	14550 6100 14600 6100
 Text HLabel 14600 4400 2    50   Output ~ 0
 SR_CLK
@@
 NoConn ~ 3150 6300
 NoConn ~ 3150 6400
+NoConn ~ 14550 6100
 $EndSCHEMATC
