File: hardware/project/ADC_Test/ADC_Test.kicad_pcb (KiCad board)
At the start: 2 copper layers, 160 x 100 mm, 386 parts, among them J101 RF_Shield_One_Piece, J102 Conn_01x02_Male, J103 Conn_01x04_Male, J301 C64AC, J701 Conn_02x01, J702 20021111-00010T4LF, J801 Conn_01x04_Male, J802 Conn_02x05, K601 HE3621A0510, K602 HE3621A0510, K603 HE3621A0510, Q201 BC847, Q501 BC847, Q601 BC847, Q602 BC857, Q801 BC857, U201 LT8330_S6, U202 LT8330_S6, U203 TSR1-2490, U204 LM1117DTX-5.0/NOPB, U205 LT3030, U206 LM317_TO-263, U207 LM337_TO263, U208 TSR1-2450, U209 LT8330_S6, U210 LM1117DTX-3.3/NOPB, U211 LM337_TO263, U401 LAN8742A, U402 LC03-3.3, U403 LC03-3.3, U501 DG211B, U502 OPA2192, U503 DG419xY, U504 LT5400-100k-100k, U505 LM399H, U506 LT5400-5k-1k, U507 OPA177, U508 OPA140, U509 OPA177, U510 OPA192, U511 LT5400-10k-10k, U512 LM311, U601 DG211B, U602 DG211B, U603 SN74LVC1T45DBV, U604 SN74LVC1T45DBV, U605 SN74LVC1T45DBV, U606 74HCT595, U607 74HCT595, U608 LTC1052, U609 AD711, U610 AD711, U611 TL431DBZ, U612 TL431DBZ, U613 LT5400-9k-1k, U701 STM32H743ZI/STM32F765ZGT6, U702 24LC08B-E/MS, U801 SN74LVC1T45DBV, U802 SN74LVC1T45DBV, U803 ICE40HX4K-TQ144, U804 SN74LVC1T45DBV, U805 SN74LVC1T45DBV, U806 SN74LVC1T45DBV, U807 SN74LVC1T45DBV, U808 ASDMB-100.000MHZ, U809 MT25QL128ABA1ESE, Y401 NX5032GA-25.000M-LN-CD-1, Y701 NX3225GD-8MHZ-STD-CRA-3

Commit message: Changes in documentation, schematics and PCB.
Parts:
- added R523: DNP, Resistor_SMD:R_0603_1608Metric_Pad1.05x0.95mm_HandSolder, F.Cu at (-12.2, 78.2)
- C207, C212, C213, C229, C235, C242, C401, C402, C403, C404, C405, C408, C410, C412, C413, C414, C701, C702, C703, C704, C705, C706, C707, C708, C709, C710, C711, C712, C713, C714, C715, C716, C717, C718, C719, C720, C721, FB401, FB701, R406, R407, R408, R409, R411, R412, R413, R414, R415, R416, R417, R418, R419, R420, R421, R701, R702, R703, R704, R705, R706, R707, R708, U809, Y701: moved to B.Cu
- moved FB701 310.5 mm to (168.1, 118.7), turned to 180 degrees
- moved C709 300.0 mm to (154.6, 98.6), turned to 270 degrees
- moved C705 292.8 mm to (170.1, 113.4), turned to 90 degrees
- moved C703 291.3 mm to (168.7, 107.2), turned to 180 degrees
- moved R701 289.1 mm to (165.2, 119.8), turned to 270 degrees
- moved U702 287.9 mm to (167.5, 91.4)
- moved Y701 287.6 mm to (164.1, 113.4)
- moved C702 286.3 mm to (168.7, 102.2), turned to 180 degrees
- moved C714 285.8 mm to (167.4, 113.4), turned to 90 degrees
- moved D702 284.8 mm to (146.9, 118.2), turned to 90 degrees
- moved D703 283.1 mm to (149.6, 118.2), turned to 90 degrees
- moved C715 283.1 mm to (166.0, 95.2)
- moved C707 283.0 mm to (169.7, 98.6), turned to 270 degrees
- moved R708 283.0 mm to (155.8, 91.2), turned to 90 degrees
- moved R706 281.9 mm to (166.8, 98.6), turned to 90 degrees
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Other:
- copper layers 2 -> 4
- net class Default: clearance 0.2 -> 0.127; trace_width 0.25 -> 0.127; via_dia 0.8 -> 0.5; via_drill 0.4 -> 0.2
- rule pad_to_mask_clearance: 0.05 -> 0
- rule trace_clearance: 0.2 -> 0.127
- rule trace_min: 0.2 -> 0.127
- rule via_min_drill: 0.3 -> 0.2
- rule via_min_size: 0.4 -> 0.2

Commit message: PCB design
Parts:
- removed the C811 at (116.5, 169.0)
- removed the C826 at (120.1, 174.3)
- removed the J102 at (146.9, 110.5)
- removed the J701 at (158.9, 120.0)
- removed the R523 at (-12.2, 78.2)
- removed the R701 at (165.2, 119.8)
- removed the R812 at (111.4, 174.0)
- added C501: 10p, Capacitor_SMD:C_0603_1608Metric_Pad1.05x0.95mm_HandSolder, B.Cu at (106.4, 52.5)
- added D501: 1N4148W, Diode_SMD:D_SOD-123, F.Cu at (105.7, 49.1)
- added D502: BZT585B15TQ-13, Diode_SMD:D_SOD-523, F.Cu at (131.1, -4.71)
- added K501: 9012, ADC_TEST:9012, F.Cu at (110.0, 52.1)
- added Q501: BC847, Package_TO_SOT_SMD:SOT-23, F.Cu at (105.7, 54.1)
- added Q502: MMBTA55, Package_TO_SOT_SMD:SOT-23, F.Cu at (119.1, 54.5)
- added R501: 10k, Resistor_SMD:R_0603_1608Metric_Pad1.05x0.95mm_HandSolder, B.Cu at (104.9, 52.5)
- added R502: 4k7/.1%, Resistor_SMD:R_0603_1608Metric_Pad1.05x0.95mm_HandSolder, F.Cu at (116.6, 54.5)
- added R504: 4k7/.1%, Resistor_SMD:R_0603_1608Metric_Pad1.05x0.95mm_HandSolder, F.Cu at (122.4, 54.5)
- added R506: 0, Resistor_SMD:R_0603_1608Metric_Pad1.05x0.95mm_HandSolder, F.Cu at (99.2, 47.6)
- added R508: 0, Resistor_SMD:R_0603_1608Metric_Pad1.05x0.95mm_HandSolder, F.Cu at (87.1, 13.7)
- added U504: LT1021-7, Package_SO:SOIC-8_3.9x4.9mm_P1.27mm, F.Cu at (119.5, 49.5)
- C205, C208, C209, C210, C211, C214, C215, C216, C217, C218, C219, C220, C222, C223, C224, C225, C233, C234, C236, C237, C238, C239, C240, C241, C243, C244, C245, C246, C507, C524, D201, D202, D203, D803, R206, R209, R211, R213, R214, R215, R216, R217, R218, R220, R226, R227, R228, R801, R807, R810, R811, U808: moved to B.Cu
- C502: renamed from C501; moved to B.Cu
- C505: renamed from C504; moved to B.Cu
- C506: renamed from C505; moved to B.Cu
- C510: renamed from C512; moved to B.Cu
- C514: renamed from C516; moved to B.Cu
- C516: renamed from C509; moved to B.Cu
- C519: renamed from C520; moved to B.Cu
- C521: renamed from C523; moved to B.Cu
- C522: renamed from C515; moved to B.Cu
- C523: renamed from C517; moved to B.Cu
- C801: renamed from C802; moved to B.Cu
- C802: renamed from C804; moved to B.Cu
- C803: renamed from C806; moved to B.Cu
- C804: renamed from C808; moved to B.Cu
- C805: renamed from C809; moved to B.Cu
- C806: renamed from C810; moved to B.Cu
- C807: renamed from C812; moved to B.Cu
- C808: renamed from C813; moved to B.Cu
- C809: renamed from C814; moved to B.Cu
- C810: renamed from C815; moved to B.Cu
- C811: renamed from C816; moved to B.Cu
- C812: renamed from C817; moved to B.Cu
- C813: renamed from C818; moved to B.Cu
- C814: renamed from C819; moved to B.Cu
- C815: renamed from C820; moved to B.Cu
- C816: renamed from C821; moved to B.Cu
- C817: renamed from C822; moved to B.Cu
- C818: renamed from C823; moved to B.Cu
- C819: renamed from C824; moved to B.Cu
- C820: renamed from C825; moved to B.Cu
- C821: renamed from C801; moved to B.Cu
- C822: renamed from C803; moved to B.Cu
- C823: renamed from C827; moved to B.Cu
- C824: renamed from C805; moved to B.Cu
- C825: renamed from C828; moved to B.Cu
- C826: renamed from C807; moved to B.Cu
- C827: renamed from C829; moved to B.Cu
- C828: renamed from C830; moved to B.Cu
- C829: renamed from C831; moved to B.Cu
- C830: renamed from C832; moved to B.Cu
- D505: renamed from D503; moved to B.Cu
- J101: value RF_Shield_One_Piece -> Conn_01x03_Male; footprint ADC_TEST:36107406S -> Connector_PinHeader_2.54mm:PinHeader_1x03_P2.54mm_Vertical
- R523: renamed from R518; moved to B.Cu
- R812: renamed from R813; moved to B.Cu
- R813: renamed from R814; moved to B.Cu
- R814: renamed from R815; moved to B.Cu
- R815: renamed from R816; moved to B.Cu
- R816: renamed from R817; moved to B.Cu
- R817: renamed from R818; moved to B.Cu
- R818: renamed from R819; moved to B.Cu
- R819: renamed from R820; moved to B.Cu
- moved Q201 311.0 mm to (266.7, 55.6), turned to 180 degrees
- moved J101 289.6 mm to (152.8, 114.4)
- moved C206 271.3 mm to (270.3, 54.6), turned to 180 degrees
- moved R201 270.6 mm to (270.3, 56.6)
- moved R621 267.8 mm to (251.6, 76.2), turned to 90 degrees
- moved C205 267.5 mm to (215.3, 127.4), turned to 90 degrees
- moved R603 265.3 mm to (232.0, 18.7)
- moved R602 262.9 mm to (235.8, 18.7)
- moved R608 262.8 mm to (235.8, 25.5), turned to 180 degrees
- moved R611 262.2 mm to (238.6, 84.3), turned to 270 degrees
- moved R221 260.6 mm to (188.5, 124.1)
- moved R609 255.2 mm to (239.6, 25.5), turned to 180 degrees
- moved R222 254.7 mm to (188.6, 131.3)
- moved C225 253.1 mm to (215.3, 117.2), turned to 90 degrees
- moved R613 251.1 mm to (241.7, 84.3), turned to 270 degrees
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- renumbered C502 to C503, C503 to C504, C510 to C508, C511 to C509, C513 to C511, C506 to C512, C514 to C513, C508 to C515, C518 to C517, C519 to C518, C521 to C520, C522 to C525, D501 to D503, D502 to D504, J103 to J102, J702 to J701, Q501 to Q503, R501 to R503, R502 to R505, R503 to R507, R504 to R509, R505 to R510, R506 to R511, R507 to R512, R508 to R513, R509 to R514, R510 to R515, R511 to R516, R512 to R517, R513 to R518, R514 to R519, R515 to R520, R516 to R521, R517 to R522, R519 to R524, R520 to R525, R521 to R526, R522 to R527, R702 to R701, R703 to R702, R704 to R703, R705 to R704, R706 to R705, R707 to R706, R708 to R707, U504 to U505, U505 to U506, U506 to U507, U507 to U508, U508 to U509, U509 to U510, U510 to U511, U511 to U512, U512 to U513
Connections:
- J101 pad 1: AGNDF -> /FPGA/FPGA_UART2_TX_TTL
- L202 pad 2: Net-(C211-Pad2) -> Net-(C210-Pad1)
- L202 pad 3: +24VF -> AGNDF
- L203 pad 1: AGNDF -> +24VF
- L203 pad 4: Net-(C210-Pad1) -> Net-(C211-Pad2)
- U701 pad 34: /MCU/MCU_DEFAULT -> (no net)
- U803 pad 39: (no net) -> /ADC/FPGA_AD_RFS_OPT
- U803 pad 61: /FPGA/100MHZ_OPT -> (no net)
Routing:
- net +3.3VF: track 0.00 -> 78.2 mm, vias 0 -> 32
- net +3.3VP: track 0.00 -> 44.8 mm, vias 0 -> 21
- net Net-(C515-Pad2): track 0.00 -> 41.3 mm, vias 0 -> 1
- net Net-(K501-Pad4): track 0.00 -> 40.4 mm
- net AGNDF: track 0.00 -> 39.5 mm, vias 0 -> 20
- net /Ethernet/NRST: track 0.00 -> 39.0 mm, vias 0 -> 1
- net -14VF: track 0.00 -> 38.7 mm, vias 0 -> 17
- net /FPGA/iCE_MISO: track 0.00 -> 36.3 mm, vias 0 -> 1
- net /FPGA/iCE_SCK: track 0.00 -> 36.0 mm, vias 0 -> 1
- net /FPGA/iCE_SS_B: track 0.00 -> 32.5 mm, vias 0 -> 1
- net /FPGA/iCE_MOSI: track 0.00 -> 32.1 mm, vias 0 -> 1
- net Net-(C515-Pad1): track 0.00 -> 31.6 mm, vias 0 -> 1
- net /FPGA/iCE_CRESET: track 0.00 -> 27.6 mm, vias 0 -> 2
- net +18VF: track 0.00 -> 20.9 mm, vias 0 -> 17
- net +5VF: track 0.00 -> 20.3 mm, vias 0 -> 9
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- added copper zone on B.Cu, net +18VF
- added copper zone on F.Cu, net +18VF
- added copper zone on Power, net +1V2
- added copper zone on B.Cu, net +24VF
- added copper zone on F.Cu, net +24VF
- added copper zone on Power, net +24VF
- added copper zone on B.Cu, net +3.3VF
- added copper zone on F.Cu, net +3.3VF
- added copper zone on Power, net +3.3VF
- added copper zone on Power, net +3.3VP
- added copper zone on B.Cu, net +5VF
- added copper zone on F.Cu, net +5VF
- added copper zone on Power, net +5VF
- added copper zone on B.Cu, net -14VF
- added copper zone on F.Cu, net -14VF
- added copper zone on Power, net -14VF
- added copper zone on B.Cu, net -18VF
- added copper zone on F.Cu, net -18VF
- added copper zone on Power, net -18VF
- added copper zone on B.Cu, net AGNDF
- added copper zone on F.Cu, net AGNDF
- added copper zone on Ground, net AGNDF
- added copper zone on B.Cu, net Net-(C211-Pad1)
- added copper zone on F.Cu, net Net-(C211-Pad1)
- added copper zone on B.Cu, net Net-(C211-Pad2)
- added copper zone on F.Cu, net Net-(C211-Pad2)
- added copper zone on F.Cu, net Net-(C212-Pad1)
- added copper zone on Power, net Net-(C212-Pad1)
- added copper zone on B.Cu, net Net-(C216-Pad1)
- added copper zone on F.Cu, net Net-(C216-Pad1)
- added copper zone on B.Cu, net Net-(C239-Pad1)
- added copper zone on F.Cu, net Net-(C239-Pad1)
- added copper zone on B.Cu, net Net-(C239-Pad2)
- added copper zone on F.Cu, net Net-(C239-Pad2)
- added copper zone on B.Cu, net Net-(C243-Pad1)
- added copper zone on F.Cu, net Net-(C243-Pad1)
- added copper zone on Power, net Net-(C243-Pad1)
- added copper zone on B.Cu, net Net-(R214-Pad1)
- added copper zone on F.Cu, net Net-(R214-Pad1)
- added copper zone on B.Cu, net Net-(R227-Pad1)
- added copper zone on F.Cu, net Net-(R227-Pad1)
- added copper zone on Power, net VCCQ
Other:
- outline, holes or cut-outs redrawn
- board text added: "J101"
- board text added: "J102"
- board text added: "SPI MISO"
- board text added: "SPI MOSI"
- board text added: "SPI SCK"
- board text added: "SPI nSS"
- board text added: "UART CTRL"
- board text added: "UART RX"
- board text added: "UART TX"

Commit message: PCB design.
Parts:
- removed the C206 at (270.3, 54.6)
- removed the C509 at (138.6, -53.7)
- removed the C615 at (208.4, 23.2)
- removed Q201: BC847, Package_TO_SOT_SMD:SOT-23
- removed the R201 at (270.3, 56.6)
- removed the R206 at (197.2, 131.6)
- removed TP501, TP502, TP503: TestPoint, TestPoint:TestPoint_Loop_D2.60mm_Drill1.6mm_Beaded
- C508, C601, C614, D502, R508, R615, R616, R617, R618, U702: moved to B.Cu
- C516: renamed from C517; moved to B.Cu
- C517: renamed from C518; moved to B.Cu
- C602: renamed from C603; moved to B.Cu
- C603: renamed from C602; moved to B.Cu
- C604: renamed from C606; moved to B.Cu
- C605: renamed from C604; moved to B.Cu
- C606: renamed from C608; moved to B.Cu
- C607: renamed from C605; moved to B.Cu
- C608: renamed from C611; moved to B.Cu
- C609: renamed from C607; moved to B.Cu
- C611: renamed from C613; moved to B.Cu
- C612: renamed from C609; moved to B.Cu
- C613: renamed from C612; moved to B.Cu
- C615: renamed from C616; moved to B.Cu
- C616: renamed from C617; moved to B.Cu
- C617: renamed from C618; moved to B.Cu
- C618: renamed from C619; moved to B.Cu
- C619: renamed from C620; moved to B.Cu
- C620: renamed from C621; moved to B.Cu
- C621: renamed from C622; moved to B.Cu
- C622: renamed from C623; moved to B.Cu
- C623: renamed from C624; moved to B.Cu
- C625: renamed from C626; moved to B.Cu
- moved C517 125.2 mm to (160.5, 65.0)
- moved C508 105.3 mm to (122.4, 54.5), turned to 90 degrees
- moved R513 104.2 mm to (134.9, 60.8), turned to 270 degrees
- moved C614 98.7 mm to (167.3, 96.4), turned to 180 degrees
- moved R601 98.3 mm to (213.0, 66.4), turned to 90 degrees
- moved C608 95.9 mm to (171.3, 98.7), turned to 180 degrees
- moved R619 94.5 mm to (200.7, 70.2)
- moved L601 94.4 mm to (200.7, 67.3)
- moved R620 93.7 mm to (196.8, 67.3), turned to 0 degrees
- moved R610 93.5 mm to (193.2, 74.9), turned to 180 degrees
- moved R617 93.1 mm to (170.1, 85.0), turned to 270 degrees
- moved C609 91.8 mm to (171.3, 96.4), turned to 180 degrees
- moved R628 90.6 mm to (154.4, 59.4), turned to 180 degrees
- moved C611 90.3 mm to (167.3, 98.7), turned to 180 degrees
- moved Q601 89.6 mm to (161.5, 53.6), turned to 90 degrees
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- renumbered C207 to C206, C208 to C207, C209 to C208, C210 to C209, C211 to C210, C212 to C211, C213 to C212, C214 to C213, C215 to C214, C216 to C215, C217 to C216, C218 to C217, C219 to C218, C220 to C219, C221 to C220, C222 to C221, C223 to C222, C224 to C223, C225 to C224, C226 to C225, C227 to C226, C228 to C227, C229 to C228, C230 to C229, C231 to C230, C232 to C231, C233 to C232, C234 to C233, C235 to C234, C236 to C235, C237 to C236, C238 to C237, C239 to C238, C240 to C239, C241 to C240, C242 to C241, C243 to C242, C244 to C243, C245 to C244, C246 to C245, C510 to C509, C511 to C510, C512 to C511, C513 to C512, C514 to C513, C515 to C514, C516 to C515, C519 to C518, C520 to C519, C521 to C520, C522 to C521, C523 to C522, C524 to C523, C525 to C524, C625 to C624, R202 to R201, R203 to R202, R204 to R203, R205 to R204, R207 to R205, R208 to R206, R209 to R207, R210 to R208, R211 to R209, R212 to R210, R213 to R211, R214 to R212, R215 to R213, R216 to R214, R217 to R215, R218 to R216, R219 to R217, R220 to R218, R221 to R219, R222 to R220, R223 to R221, R224 to R222, R225 to R223, R226 to R224, R227 to R225, R228 to R226, R704 to R701, R705 to R702, R706 to R703, R701 to R704, R702 to R705, R703 to R706, R809 to R801, R805 to R802, R804 to R803, R803 to R804, R802 to R805, R801 to R807, R807 to R809
Connections:
- C211 pad 1: Net-(C212-Pad1) -> Net-(C211-Pad1)
- C212 pad 1: Net-(C212-Pad1) -> Net-(C211-Pad1)
- Q801 pad 2: +3.3VF -> +3.3VP
- R205 pad 1: Net-(C212-Pad1) -> Net-(C211-Pad1)
- R210 pad 1: Net-(C212-Pad1) -> Net-(C211-Pad1)
- R704 pad 1: Net-(R701-Pad1) -> Net-(R704-Pad1)
- R705 pad 1: Net-(R702-Pad1) -> Net-(R705-Pad1)
- R706 pad 1: Net-(R703-Pad1) (its old number) -> Net-(R706-Pad1)
- R801 pad 2: Net-(R809-Pad2) -> Net-(R801-Pad2)
- R802 pad 1: Net-(R805-Pad1) -> Net-(R802-Pad1)
- R803 pad 1: Net-(R804-Pad1) -> Net-(R803-Pad1)
- R804 pad 1: Net-(R803-Pad1) -> Net-(R804-Pad1)
- R805 pad 1: Net-(R802-Pad1) -> Net-(R805-Pad1)
- R807 pad 1: Net-(R801-Pad1) -> Net-(R807-Pad1)
- R809 pad 1: Net-(R807-Pad1) -> Net-(R809-Pad1)
- U203 pad 3: Net-(C212-Pad1) -> Net-(C211-Pad1)
- U204 pad 3: Net-(C212-Pad1) -> Net-(C211-Pad1)
- U205 pad 11: /Power/~SHDN -> Net-(C211-Pad1)
- U205 pad 13: Net-(C212-Pad1) -> Net-(C211-Pad1)
- U205 pad 14: Net-(C212-Pad1) -> Net-(C211-Pad1)
- U205 pad 17: Net-(C212-Pad1) -> Net-(C211-Pad1)
- U205 pad 18: Net-(C212-Pad1) -> Net-(C211-Pad1)
- U205 pad 20: /Power/~SHDN -> Net-(C211-Pad1)
- U701 pad 1: /Input/SR_LAT -> Net-(R704-Pad1)
- U701 pad 115: (no net) -> /FPGA/FPGA_IO3
- U701 pad 116: (no net) -> /FPGA/FPGA_IO4
- U701 pad 2: /Input/SR_DAT -> Net-(R705-Pad1)
- U701 pad 3: /Input/SR_CLK -> Net-(R706-Pad1)
- U701 pad 68: /MCU/FGPA_PWR_ON -> (no net)
- U701 pad 7: Net-(R701-Pad1) -> (no net)
- U701 pad 76: (no net) -> /Input/SR_LAT
- U701 pad 8: Net-(R702-Pad1) -> (no net)
- U701 pad 86: (no net) -> /Input/SR_CLK
- U701 pad 9: Net-(R703-Pad1) (its old number) -> (no net)
- U701 pad 92: (no net) -> /Input/SR_DAT
- U803 pad 1: Net-(R802-Pad1) -> Net-(R801-Pad2)
- U803 pad 10: Net-(R807-Pad1) -> (no net)
- U803 pad 101: /FPGA/FPGA_IO2 -> /FPGA/FPGA_IO4
- U803 pad 102: /FPGA/FPGA_IO1 -> /FPGA/FPGA_IO3
- U803 pad 104: (no net) -> /FPGA/FPGA_SPI3_MOSI
- U803 pad 105: (no net) -> /FPGA/FPGA_SPI3_MISO
- U803 pad 106: (no net) -> /FPGA/FPGA_SPI3_SCK
- U803 pad 107: (no net) -> /FPGA/FPGA_SPI3_NSS
- U803 pad 110: Net-(J801-Pad1) -> Net-(R802-Pad1)
- U803 pad 112: Net-(J801-Pad2) -> (no net)
- U803 pad 113: Net-(J801-Pad3) -> (no net)
- U803 pad 114: Net-(J801-Pad4) -> (no net)
- U803 pad 115: (no net) -> Net-(R803-Pad1)
- U803 pad 121: (no net) -> Net-(R804-Pad1)
- U803 pad 130: (no net) -> Net-(R805-Pad1)
- U803 pad 136: (no net) -> Net-(R806-Pad1)
- U803 pad 2: Net-(R803-Pad1) -> Net-(J801-Pad1)
- U803 pad 3: Net-(R804-Pad1) -> Net-(J801-Pad2)
- U803 pad 37: Net-(R809-Pad2) -> Net-(R807-Pad1)
- U803 pad 38: (no net) -> Net-(R809-Pad1)
- U803 pad 39: /ADC/FPGA_AD_RFS_OPT -> (no net)
- U803 pad 4: Net-(R805-Pad1) -> Net-(J801-Pad3)
- U803 pad 7: Net-(R806-Pad1) -> Net-(J801-Pad4)
- U803 pad 73: /FPGA/FPGA_SPI3_SCK -> (no net)
- U803 pad 8: (no net) -> /ADC/FPGA_AD_RFS_OPT
- U803 pad 81: (no net) -> /FPGA/FPGA_UART2_CTRL_TTL
- U803 pad 82: (no net) -> /FPGA/FPGA_UART2_RX_TTL
- U803 pad 83: (no net) -> /FPGA/FPGA_UART2_TX_TTL
- U803 pad 9: Net-(R801-Pad1) -> (no net)
- U803 pad 91: /FPGA/FPGA_SPI3_NSS -> (no net)
- U803 pad 95: /FPGA/FPGA_SPI3_MISO -> (no net)
- U803 pad 96: /FPGA/FPGA_SPI3_MOSI -> (no net)
- U803 pad 97: /FPGA/FPGA_UART2_RX_TTL -> (no net)
- U803 pad 98: /FPGA/FPGA_UART2_CTRL_TTL -> /FPGA/FPGA_IO2
- U803 pad 99: /FPGA/FPGA_UART2_TX_TTL -> /FPGA/FPGA_IO1
Routing:
- net AGNDF: track 39.5 -> 305.6 mm, vias 20 -> 48
- net /ADC/FPGA_AD_RFS_OPT: track 0.00 -> 75.2 mm, vias 0 -> 1
- net /Input/K2_CTR: track 0.00 -> 65.1 mm, vias 0 -> 1
- net Net-(R623-Pad2): track 0.00 -> 62.5 mm, vias 0 -> 2
- net /ADC/FPGA_AD_RFS: track 0.00 -> 61.2 mm, vias 0 -> 2
- net /Input/K1_CTR: track 0.00 -> 54.1 mm, vias 0 -> 1
- net /Input/K3_CTR: track 0.00 -> 45.0 mm, vias 0 -> 1
- net /ADC/ADIN: track 0.00 -> 39.8 mm, vias 0 -> 1
- net +5VF: track 20.3 -> 57.3 mm, vias 9 -> 25
- net Net-(K601-Pad4): track 0.51 -> 37.2 mm
- net /FPGA/FGPA_AD_VRH: track 0.00 -> 35.3 mm, vias 0 -> 2
- net /FPGA/iCE_CDONE: track 2.16 -> 34.6 mm
- net /ADC/FGPA_AD_ID: track 0.00 -> 31.9 mm, vias 0 -> 2
- net /ADC/FGPA_AD_IRP: track 0.00 -> 31.0 mm, vias 0 -> 2
- net /Connector/V_HIGH: track 0.00 -> 30.5 mm
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- added copper zone on B.Cu, net Net-(C211-Pad1)
- added copper zone on F.Cu, net Net-(C211-Pad1)
- added copper zone on Power, net Net-(C211-Pad1)
- added copper zone on B.Cu, net Net-(C216-Pad1)
- added copper zone on B.Cu, net Net-(C243-Pad1)
- added copper zone on Power, net Net-(C243-Pad1)
- added copper zone on F.Cu, net Net-(Q601-Pad1)
- added copper zone on F.Cu, net Net-(Q602-Pad1)
- added copper zone on F.Cu, net Net-(R627-Pad1)
- added copper zone on F.Cu, net Net-(R628-Pad2)
- added copper zone on B.Cu, net VCC
- added copper zone on F.Cu, net VCC
- added copper zone on Power, net VCC
- added copper zone on B.Cu, net VDD
- added copper zone on F.Cu, net VDD
- added copper zone on Power, net VDD
- removed copper zone on B.Cu, net Net-(C210-Pad1)
- removed copper zone on F.Cu, net Net-(C210-Pad1)
- removed copper zone on F.Cu, net Net-(C212-Pad1)
- removed copper zone on Power, net Net-(C212-Pad1)
- removed copper zone on Power, net Net-(C242-Pad1)
Other:
- outline, holes or cut-outs redrawn

Commit message: PCB layout almost done.
Parts:
- moved C401 3.68 mm to (185.2, 93.3)
- moved C404 3.43 mm to (189.0, 93.3)
- moved C708 2.25 mm to (178.1, 102.5), turned to 90 degrees
- moved C519 1.35 mm to (122.0, 61.2)
- moved R515 1.35 mm to (122.0, 65.2)
- moved C516 1.35 mm to (125.5, 60.6)
- moved U510 1.35 mm to (126.5, 63.1)
- moved R521 1.35 mm to (130.9, 65.0)
- moved R513 1.35 mm to (134.0, 61.8)
- moved R516 1.35 mm to (130.9, 61.2)
- moved D202 1.09 mm to (88.0, 75.3)
- moved C224 0.76 mm to (215.3, 116.5)
- moved C510 0.76 mm to (142.0, 82.5)
- moved R207 0.76 mm to (74.7, 73.7)
- moved R512 0.76 mm to (144.4, 82.5)
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Routing:
- net +5VF: track 57.3 -> 240.3 mm, vias 25 -> 29
- net -18VF: track 10.6 -> 165.0 mm, vias 10 -> 11
- net (no net): track 0.00 -> 117.3 mm
- net Net-(R628-Pad2): track 28.4 -> 140.5 mm, vias 3 -> 4
- net Net-(C511-Pad1): track 4.83 -> 64.3 mm
- net -14VF: track 63.0 -> 106.1 mm, vias 24 -> 26
- net /Ethernet/RMII_CRS_DV: track 0.00 -> 41.6 mm
- net /Ethernet/RMII_MDIO: track 4.94 -> 46.5 mm, vias 0 -> 2
- net /Ethernet/REF_CLK: track 0.00 -> 41.5 mm
- net /Ethernet/RMII_RXD0: track 0.00 -> 41.5 mm
- net /Ethernet/RMII_MDC: track 0.00 -> 41.5 mm, vias 0 -> 1
- net /Ethernet/RMII_TXD1: track 0.00 -> 41.5 mm, vias 0 -> 2
- net AGNDF: track 305.6 -> 346.9 mm, vias 48 -> 88
- net /Ethernet/RMII_TXD0: track 0.00 -> 40.5 mm, vias 0 -> 2
- net /Ethernet/RMII_TXEN: track 0.00 -> 39.4 mm, vias 0 -> 2
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- added copper zone on Power, net +18VF
- added copper zone on B.Cu, net +1V2
- added copper zone on F.Cu, net +1V2
- added copper zone on B.Cu, net +3.3VP
- added copper zone on F.Cu, net +3.3VP
- added copper zone on B.Cu, net Earth
- added copper zone on F.Cu, net Earth
- added copper zone on Ground, net Earth
- added copper zone on Power, net Earth
- added copper zone on B.Cu, net Net-(C206-Pad1)
- added copper zone on F.Cu, net Net-(C206-Pad1)
- added copper zone on B.Cu, net Net-(C209-Pad1)
- added copper zone on F.Cu, net Net-(C209-Pad1)
- added copper zone on B.Cu, net Net-(C209-Pad2)
- added copper zone on F.Cu, net Net-(C209-Pad2)
- added copper zone on B.Cu, net Net-(C210-Pad1)
- added copper zone on F.Cu, net Net-(C210-Pad1)
- added copper zone on B.Cu, net Net-(C214-Pad1)
- added copper zone on F.Cu, net Net-(C214-Pad1)
- added copper zone on Power, net Net-(C215-Pad1)
- added copper zone on F.Cu, net Net-(C220-Pad1)
- added copper zone on F.Cu, net Net-(C221-Pad1)
- added copper zone on B.Cu, net Net-(C228-Pad1)
- added copper zone on F.Cu, net Net-(C228-Pad1)
- added copper zone on B.Cu, net Net-(C234-Pad1)
- added copper zone on F.Cu, net Net-(C234-Pad1)
- added copper zone on Power, net Net-(C242-Pad1)
- added copper zone on B.Cu, net Net-(C414-Pad1)
- added copper zone on B.Cu, net Net-(R211-Pad1)
- added copper zone on F.Cu, net Net-(R211-Pad1)
- removed copper zone on B.Cu, net Net-(C216-Pad1)
- removed copper zone on B.Cu, net Net-(C243-Pad1)
- removed copper zone on Power, net Net-(C243-Pad1)
Other:
- outline, holes or cut-outs redrawn
- net class +24V added: clearance 0.254, trace_width 0.127, via_dia 0.5, via_drill 0.2
- board text added: "1"
- board text added: "2"
- board text added: "24V"
- board text added: "3"
- board text added: "4"
- board text added: "ADC TEST"
- board text added: "GND"
- board text added: "RX+"
- board text added: "RX-"
- board text added: "TCP/IP 192.168.1.123:2000"
- board text added: "TX+"
- board text added: "TX-"
- board text added: "V+"
- board text added: "V-"

Commit message: PCB design done.
Parts:
- R515: value 1k96/.1% -> 3k01/.1%
- R517: value 62k6/.1% -> 62k
- R520: value 400/.1% -> 0
Connections:
- C524 pad 1: +3.3VF -> +3.3VP
- R525 pad 1: +3.3VF -> +3.3VP
- U505 pad 1: /ADC/ADIN -> Net-(U505-Pad1)
- U505 pad 2: Net-(U505-Pad2) -> Net-(U505-Pad1)
- U505 pad 8: Net-(U505-Pad2) -> /ADC/ADIN
- U513 pad 8: +3.3VF -> +3.3VP
Routing:
- net +3.3VP: track 51.2 -> 90.3 mm, vias 27 -> 29
- net AGNDF: track 346.9 -> 356.8 mm, vias 88 -> 94
- net Net-(U505-Pad2): track 5.42 -> 0.00 mm
- net /ADC/ADIN: track 39.8 -> 44.7 mm
- net +3.3VF: track 91.2 -> 86.7 mm, vias 38 -> 36
- net Net-(C221-Pad1): track 11.0 -> 13.2 mm
- net Net-(U505-Pad1): track 0.00 -> 0.65 mm
Other:
- outline, holes or cut-outs redrawn

Commit message: MCU readout from FPGA works.
Connections:
- net /Input/K3_CTR renamed /Input/K4_CTR
