File: hardware/project/ADC_Test/ADC_Test.kicad_pcb (KiCad board)
At the start: 4 copper layers, 160 x 100 mm, 383 parts, among them J101 Conn_01x03_Male, J102 Conn_01x04_Male, J301 C64AC, J701 20021111-00010T4LF, J801 Conn_01x04_Male, J802 Conn_02x05, K501 9012, K601 HE3621A0510, K602 HE3621A0510, K603 HE3621A0510, Q501 BC847, Q502 MMBTA55, Q503 BC847, Q601 BC847, Q602 BC857, Q801 BC857, U201 LT8330_S6, U202 LT8330_S6, U203 TSR1-2490, U204 LM1117DTX-5.0/NOPB, U205 LT3030, U206 LM317_TO-263, U207 LM337_TO263, U208 TSR1-2450, U209 LT8330_S6, U210 LM1117DTX-3.3/NOPB, U211 LM337_TO263, U401 LAN8742A, U402 LC03-3.3, U403 LC03-3.3, U501 DG211B, U502 OPA2192, U503 DG419xY, U504 LT1021-7, U505 LT5400-100k-100k, U506 LM399H, U507 LT5400-5k-1k, U508 OPA177, U509 OPA140, U510 OPA177, U511 OPA192, U512 LT5400-10k-10k, U513 LM311, U601 DG211B, U602 DG211B, U603 SN74LVC1T45DBV, U604 SN74LVC1T45DBV, U605 SN74LVC1T45DBV, U606 74HCT595, U607 74HCT595, U608 LTC1052, U609 AD711, U610 AD711, U611 TL431DBZ, U612 TL431DBZ, U613 LT5400-9k-1k, U701 STM32H743ZI/STM32F765ZGT6, U702 24LC08B-E/MS, U801 SN74LVC1T45DBV, U802 SN74LVC1T45DBV, U803 ICE40HX4K-TQ144, U804 SN74LVC1T45DBV, U805 SN74LVC1T45DBV, U806 SN74LVC1T45DBV, U807 SN74LVC1T45DBV, U808 ASDMB-100.000MHZ, U809 MT25QL128ABA1ESE, Y401 NX5032GA-25.000M-LN-CD-1, Y701 NX3225GD-8MHZ-STD-CRA-3

Commit message: MCU sofware development.
Routing:
- net AGNDF: track 356.8 -> 398.7 mm, vias 94 -> 118
- net -14VF: track 106.1 -> 94.2 mm, vias 26 -> 25
- net +18VF: track 65.4 -> 68.8 mm, vias 27 -> 25
- net -18VF: track 165.0 -> 164.1 mm
- net /Input/K1_CTR: track 54.1 -> 54.7 mm
- net /Input/K2_CTR: track 65.1 -> 65.6 mm
- net /Input/K4_CTR: track 45.0 -> 45.5 mm
